File: Hardware/pressure sensor adapter/PressureSensorAdaptor.sch (EAGLE design)
At the start: 11 parts, among them IC1 RCV420P

Commit message: routed alternet Pressure sense adapter board
Connections:
- removed net VIN: JP3.5, U$3.VIN+, U1.EN, U1.IN
- new net 12V+: C1.1, IC1.V+, JP1.2, U$3.VO+
- new net 12V-: C2.1, IC1.V-, U$3.VO-
- net 12V: now also JP3.5, U$3.VIN+, U1.EN, U1.IN; no longer C1.1, C2.1, IC1.V+, IC1.V-, JP1.2, U$3.VO+, U$3.VO-
Other:
- note added: "Current Loop"
- moved on the sheet: C1, C2
