File: Hardware/pressure sensor adapter/PressureSensorAdaptor.sch (EAGLE design)
At the start: 12 parts, among them IC1 RCV420P

Commit message: added bulk capacitance on 12v unisolated rail
Parts:
- added C3: 10uF, SparkFun-Capacitors:CAP0805
- added C4: 0.1uf, SparkFun-Capacitors:CAP0805
- added C5: 100pF, SparkFun-Capacitors:CAP0805
- C8: value (none) -> 0.1uf
Connections:
- net 12V: now also C3.1, C4.1, C5.1
- net GND: now also C3.2, C4.2, C5.2
Changed lines of the file:
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@@
 <part name="GND-ISO4" library="SparkFun-Aesthetics" deviceset="GND-ISO" device=""/>
 <part name="SUPPLY4" library="SparkFun-Aesthetics" deviceset="5V" device=""/>
-<part name="C8" library="SparkFun-Capacitors" deviceset="CAP" device="0805"/>
+<part name="C8" library="SparkFun-Capacitors" deviceset="CAP" device="0805" value="0.1uf"/>
 <part name="GND-ISO5" library="SparkFun-Aesthetics" deviceset="GND-ISO" device=""/>
 <part name="GND-ISO6" library="SparkFun-Aesthetics" deviceset="GND-ISO" device=""/>
@@
 <attribute name="VERSION" value="A"/>
 </part>
+<part name="C3" library="SparkFun-Capacitors" deviceset="CAP" device="0805" value="10uF">
+<attribute name="DIGIKEY" value="490-3886-1-ND"/>
+</part>
+<part name="C4" library="SparkFun-Capacitors" deviceset="CAP" device="0805" value="0.1uf"/>
+<part name="C5" library="SparkFun-Capacitors" deviceset="CAP" device="0805" value="100pF"/>
+<part name="SUPPLY1" library="SparkFun-Aesthetics" deviceset="12V" device=""/>
+<part name="GND1" library="supply1" deviceset="GND" device=""/>
+<part name="GND2" library="supply1" deviceset="GND" device=""/>
+<part name="GND3" library="supply1" deviceset="GND" device=""/>
+<part name="SUPPLY2" library="SparkFun-Aesthetics" deviceset="12V" device=""/>
+<part name="SUPPLY5" library="SparkFun-Aesthetics" deviceset="12V" device=""/>
 </parts>
 <sheets>
@@
 <attribute name="DESIGNER" x="109.22" y="-132.08" size="1.016" layer="96" display="off"/>
 </instance>
+<instance part="C3" gate="G$1" x="88.9" y="-2.54">
+<attribute name="DIGIKEY" x="88.9" y="-2.54" size="1.016" layer="96" display="off"/>
+</instance>
+<instance part="C4" gate="G$1" x="81.28" y="-2.54"/>
+<instance part="C5" gate="G$1" x="73.66" y="-2.54"/>
+<instance part="SUPPLY1" gate="G$1" x="73.66" y="2.54"/>
+<instance part="GND1" gate="1" x="73.66" y="-7.62"/>
+<instance part="GND2" gate="1" x="81.28" y="-7.62"/>
+<instance part="GND3" gate="1" x="88.9" y="-7.62"/>
+<instance part="SUPPLY2" gate="G$1" x="81.28" y="2.54"/>
+<instance part="SUPPLY5" gate="G$1" x="88.9" y="2.54"/>
 </instances>
 <busses>
@@
 <wire x1="20.32" y1="0" x2="53.34" y2="0" width="0.1524" layer="91"/>
 </segment>
+<segment>
+<pinref part="C5" gate="G$1" pin="2"/>
+<pinref part="GND1" gate="1" pin="GND"/>
+</segment>
+<segment>
+<pinref part="C4" gate="G$1" pin="2"/>
+<pinref part="GND2" gate="1" pin="GND"/>
+</segment>
+<segment>
+<pinref part="C3" gate="G$1" pin="2"/>
+<pinref part="GND3" gate="1" pin="GND"/>
+</segment>
 </net>
 <net name="VOUT" class="0">
@@
 <wire x1="-63.5" y1="-27.94" x2="-63.5" y2="-25.4" width="0.1524" layer="91"/>
 </segment>
-</net>
+<segment>
+<pinref part="C5" gate="G$1" pin="1"/>
+<pinref part="SUPPLY1" gate="G$1" pin="12V"/>
+</segment>
+<segment>
+<pinref part="C4" gate="G$1" pin="1"/>
+<pinref part="SUPPLY2" gate="G$1" pin="12V"/>
+</segment>
+<segment>
+<pinref part="C3" gate="G$1" pin="1"/>
+<pinref part="SUPPLY5" gate="G$1" pin="12V"/>
+</segment>
+</net>
