File: Hardware/TestEngine1/InstrumentationBoard/InstrumentationBoard.brd (EAGLE design)
At the start: 105.1 x 80 mm, 106 parts, among them IC1 MAX31855, J1 1X2-3.5MM, Q1 MOSFET-NCHANNELBSS123LT1G, Q2 MOSFET-NCHANNELBSS123LT1G, Q3 MOSFET-NCHANNELBSS123LT1G, U1 BMP180

Commit message: work in progress
Connections:
- net GREEN: now also U$10.M0PWM5/PG1; no longer U$10.M0PWM6/PK4
- net RED: now also U$10.M0PWM6/PK4; no longer U$10.M0PWM5/PG1
Routing:
- net BLUE: track 0.00 -> 30.5 mm
- net RED: track 0.00 -> 27.2 mm
- net GREEN: track 0.00 -> 20.5 mm
- net N$7: track 0.00 -> 5.04 mm
- net N$8: track 0.00 -> 5.04 mm
- net +3V3: track 134.9 -> 138.7 mm
- net N$3: track 0.00 -> 3.25 mm
- net N$15: track 0.00 -> 2.26 mm
- net N$10: track 0.00 -> 2.26 mm
- net N$9: track 0.00 -> 2.18 mm
Changed lines of the file:
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@@
 <via x="5.715" y="27.305" extent="1-16" drill="0.6" shape="octagon"/>
 <via x="0.635" y="22.86" extent="1-16" drill="0.6" shape="octagon"/>
+<via x="69.215" y="52.07" extent="1-16" drill="0.6" shape="octagon"/>
 </signal>
 <signal name="CS">
@@
 <wire x1="70.485" y1="34.29" x2="70.485" y2="33.43" width="0.4064" layer="1"/>
 <wire x1="70.485" y1="33.43" x2="70.665" y2="33.25" width="0.4064" layer="1"/>
+<wire x1="71.755" y1="78.37" x2="75.565" y2="78.37" width="0.4064" layer="1"/>
 <wire x1="89.8" y1="76.2" x2="91.9734" y2="74.295" width="0" layer="19" extent="1-1"/>
 <wire x1="80.91" y1="77.47" x2="89.8" y2="76.2" width="0" layer="19" extent="1-1"/>
 <wire x1="75.565" y1="78.37" x2="80.91" y2="77.47" width="0" layer="19" extent="1-1"/>
 <wire x1="73.66" y1="78.37" x2="75.565" y2="78.37" width="0" layer="19" extent="1-1"/>
-<wire x1="71.755" y1="78.37" x2="73.66" y2="78.37" width="0" layer="19" extent="1-1"/>
 <wire x1="85.195" y1="40.64" x2="91.9734" y2="74.295" width="0" layer="19" extent="1-1"/>
 <wire x1="26.67" y1="25.4" x2="29.21" y2="25.4" width="0" layer="19" extent="16-16"/>
@@
 <contactref element="LED1" pad="5"/>
 <contactref element="Q3" pad="3"/>
-<wire x1="73.66" y1="67.14" x2="73.66" y2="70.39" width="0" layer="19" extent="1-1"/>
+<wire x1="73.66" y1="67.14" x2="73.66" y2="70.39" width="0.4064" layer="1"/>
 </signal>
 <signal name="N$7">
 <contactref element="LED1" pad="6"/>
 <contactref element="Q2" pad="3"/>
-<wire x1="77.47" y1="67.14" x2="75.36" y2="70.39" width="0" layer="19" extent="1-1"/>
+<wire x1="75.36" y1="70.39" x2="76.93" y2="70.39" width="0.4064" layer="1"/>
+<wire x1="76.93" y1="70.39" x2="77.47" y2="69.85" width="0.4064" layer="1"/>
+<wire x1="77.47" y1="69.85" x2="77.47" y2="67.14" width="0.4064" layer="1"/>
 </signal>
 <signal name="N$8">
 <contactref element="LED1" pad="4"/>
 <contactref element="Q1" pad="3"/>
-<wire x1="69.85" y1="67.14" x2="71.96" y2="70.39" width="0" layer="19" extent="1-1"/>
+<wire x1="71.96" y1="70.39" x2="70.39" y2="70.39" width="0.4064" layer="1"/>
+<wire x1="70.39" y1="70.39" x2="69.85" y2="69.85" width="0.4064" layer="1"/>
+<wire x1="69.85" y1="69.85" x2="69.85" y2="67.14" width="0.4064" layer="1"/>
 </signal>
 <signal name="N$9">
 <contactref element="LED1" pad="2"/>
 <contactref element="R27" pad="2"/>
-<wire x1="73.66" y1="74.39" x2="73.66" y2="76.57" width="0" layer="19" extent="1-1"/>
+<wire x1="73.66" y1="76.57" x2="73.66" y2="74.39" width="0.4064" layer="1"/>
 </signal>
 <signal name="N$10">
 <contactref element="LED1" pad="1"/>
 <contactref element="R28" pad="2"/>
-<wire x1="75.36" y1="74.39" x2="75.565" y2="76.57" width="0" layer="19" extent="1-1"/>
+<wire x1="75.36" y1="74.39" x2="75.36" y2="76.365" width="0.4064" layer="1"/>
+<wire x1="75.36" y1="76.365" x2="75.565" y2="76.57" width="0.4064" layer="1"/>
 </signal>
 <signal name="N$15">
 <contactref element="LED1" pad="3"/>
 <contactref element="R29" pad="2"/>
-<wire x1="71.96" y1="74.39" x2="71.755" y2="76.57" width="0" layer="19" extent="1-1"/>
+<wire x1="71.755" y1="76.57" x2="71.755" y2="74.595" width="0.4064" layer="1"/>
+<wire x1="71.755" y1="74.595" x2="71.96" y2="74.39" width="0.4064" layer="1"/>
 </signal>
 <signal name="BLUE">
 <contactref element="Q1" pad="1"/>
 <contactref element="R26" pad="1"/>
+<wire x1="68.9" y1="65.04" x2="68.9" y2="62.28" width="0.4064" layer="1"/>
+<wire x1="68.9" y1="62.28" x2="68.95" y2="62.23" width="0.4064" layer="1"/>
 <contactref element="U$10" pad="M0PWM7/PK5"/>
-<wire x1="68.95" y1="62.23" x2="68.9" y2="65.04" width="0" layer="19" extent="1-1"/>
-<wire x1="74.93" y1="54.61" x2="68.95" y2="62.23" width="0" layer="19" extent="1-1"/>
+<wire x1="68.95" y1="62.23" x2="68.58" y2="62.23" width="0.4064" layer="1"/>
+<wire x1="68.58" y1="62.23" x2="64.77" y2="58.42" width="0.4064" layer="1"/>
+<wire x1="74.93" y1="54.61" x2="74.93" y2="50.8" width="0.4064" layer="1"/>
+<wire x1="74.93" y1="50.8" x2="73.66" y2="49.53" width="0.4064" layer="1"/>
+<wire x1="73.66" y1="49.53" x2="67.31" y2="49.53" width="0.4064" layer="1"/>
+<wire x1="67.31" y1="49.53" x2="64.77" y2="52.07" width="0.4064" layer="1"/>
+<wire x1="64.77" y1="52.07" x2="64.77" y2="58.42" width="0.4064" layer="1"/>
 </signal>
 <signal name="GREEN">
 <contactref element="Q2" pad="1"/>
 <contactref element="R25" pad="1"/>
-<contactref element="U$10" pad="M0PWM6/PK4"/>
-<wire x1="76.57" y1="62.23" x2="76.52" y2="65.04" width="0" layer="19" extent="1-1"/>
-<wire x1="72.39" y1="54.61" x2="76.57" y2="62.23" width="0" layer="19" extent="1-1"/>
+<wire x1="76.57" y1="62.23" x2="76.57" y2="64.99" width="0.4064" layer="1"/>
+<wire x1="76.57" y1="64.99" x2="76.52" y2="65.04" width="0.4064" layer="1"/>
+<contactref element="U$10" pad="M0PWM5/PG1"/>
+<wire x1="76.57" y1="62.23" x2="76.57" y2="60.06" width="0.4064" layer="1"/>
+<wire x1="76.57" y1="60.06" x2="76.2" y2="59.69" width="0.4064" layer="1"/>
+<wire x1="76.2" y1="59.69" x2="74.295" y2="59.69" width="0.4064" layer="1"/>
+<wire x1="74.295" y1="59.69" x2="73.66" y2="59.055" width="0.4064" layer="1"/>
+<wire x1="73.66" y1="59.055" x2="68.58" y2="59.055" width="0.4064" layer="1"/>
+<wire x1="68.58" y1="59.055" x2="67.31" y2="57.785" width="0.4064" layer="1"/>
+<wire x1="67.31" y1="57.785" x2="67.31" y2="55.245" width="0.4064" layer="1"/>
+<wire x1="67.31" y1="55.245" x2="67.945" y2="54.61" width="0.4064" layer="1"/>
+<wire x1="67.945" y1="54.61" x2="69.85" y2="54.61" width="0.4064" layer="1"/>
 </signal>
 <signal name="RED">
 <contactref element="Q3" pad="1"/>
 <contactref element="R24" pad="1"/>
-<contactref element="U$10" pad="M0PWM5/PG1"/>
-<wire x1="72.76" y1="62.23" x2="72.71" y2="65.04" width="0" layer="19" extent="1-1"/>
-<wire x1="69.85" y1="54.61" x2="72.76" y2="62.23" width="0" layer="19" extent="1-1"/>
+<wire x1="72.76" y1="62.23" x2="72.76" y2="64.99" width="0.4064" layer="1"/>
+<wire x1="72.76" y1="64.99" x2="72.71" y2="65.04" width="0.4064" layer="1"/>
+<contactref element="U$10" pad="M0PWM6/PK4"/>
+<wire x1="72.76" y1="62.23" x2="72.76" y2="61.33" width="0.4064" layer="1"/>
+<wire x1="72.39" y1="54.61" x2="72.39" y2="52.07" width="0.4064" layer="1"/>
+<wire x1="72.39" y1="52.07" x2="71.12" y2="50.8" width="0.4064" layer="1"/>
+<wire x1="71.12" y1="50.8" x2="67.945" y2="50.8" width="0.4064" layer="1"/>
+<wire x1="67.945" y1="50.8" x2="66.04" y2="52.705" width="0.4064" layer="1"/>
+<wire x1="66.04" y1="52.705" x2="66.04" y2="57.785" width="0.4064" layer="1"/>
+<wire x1="66.04" y1="57.785" x2="68.58" y2="60.325" width="0.4064" layer="1"/>
+<wire x1="68.58" y1="60.325" x2="71.755" y2="60.325" width="0.4064" layer="1"/>
+<wire x1="71.755" y1="60.325" x2="72.76" y2="61.33" width="0.4064" layer="1"/>
 </signal>
 <signal name="SW_1">

Commit message: more work on board
Parts:
- moved R30 1.80 mm to (40.6, 39.4)
- moved R31 1.80 mm to (36.8, 39.4)
Changed lines of the file:
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@@
 <param name="TopRouterVariant" value="1"/>
 <param name="tpViaShape" value="round"/>
-<param name="PrefDir.1" value="a"/>
+<param name="PrefDir.1" value="|"/>
 <param name="PrefDir.2" value="0"/>
 <param name="PrefDir.3" value="0"/>
@@
 <param name="PrefDir.14" value="0"/>
 <param name="PrefDir.15" value="0"/>
-<param name="PrefDir.16" value="a"/>
+<param name="PrefDir.16" value="-"/>
 <param name="cfVia" value="8"/>
 <param name="cfNonPref" value="5"/>
@@
 <attribute name="PROD_ID" value="SWCH-08247" x="38.1" y="34.29" size="1.778" layer="27" rot="R270" display="off"/>
 </element>
-<element name="Q1" library="SparkFun-DiscreteSemi" package="SOT23-3" value="MOSFET-NCHANNELBSS123LT1G" x="69.85" y="66.04">
+<element name="Q1" library="SparkFun-DiscreteSemi" package="SOT23-3" value="MOSFET-NCHANNELBSS123LT1G" x="69.85" y="66.04" smashed="yes">
 <attribute name="PROD_ID" value="TRANS-08345" x="69.85" y="66.04" size="1.778" layer="27" display="off"/>
-</element>
-<element name="Q2" library="SparkFun-DiscreteSemi" package="SOT23-3" value="MOSFET-NCHANNELBSS123LT1G" x="77.47" y="66.04">
+<attribute name="NAME" x="69.0245" y="67.818" size="0.4064" layer="25"/>
+</element>
+<element name="Q2" library="SparkFun-DiscreteSemi" package="SOT23-3" value="MOSFET-NCHANNELBSS123LT1G" x="77.47" y="66.04" smashed="yes">
 <attribute name="PROD_ID" value="TRANS-08345" x="77.47" y="66.04" size="1.778" layer="27" display="off"/>
-</element>
-<element name="Q3" library="SparkFun-DiscreteSemi" package="SOT23-3" value="MOSFET-NCHANNELBSS123LT1G" x="73.66" y="66.04">
+<attribute name="NAME" x="76.6445" y="67.818" size="0.4064" layer="25"/>
+</element>
+<element name="Q3" library="SparkFun-DiscreteSemi" package="SOT23-3" value="MOSFET-NCHANNELBSS123LT1G" x="73.66" y="66.04" smashed="yes">
 <attribute name="PROD_ID" value="TRANS-08345" x="73.66" y="66.04" size="1.778" layer="27" display="off"/>
+<attribute name="NAME" x="72.8345" y="67.818" size="0.4064" layer="25"/>
 </element>
 <element name="R27" library="SparkFun-Resistors" package="0805" value="68" x="73.66" y="77.47" rot="R270"/>
@@
 <element name="R24" library="SparkFun-Resistors" package="0805" value="10K" x="73.66" y="62.23"/>
 <element name="R32" library="SparkFun-Resistors" package="0805" value="10K" x="41.91" y="52.07"/>
-<element name="R30" library="SparkFun-Resistors" package="0805" value="10K" x="39.37" y="38.1"/>
+<element name="R30" library="SparkFun-Resistors" package="0805" value="10K" x="40.64" y="39.37"/>
 <element name="D3" library="SparkFun-DiscreteSemi" package="SMA-DIODE" value="B340A" x="11.43" y="68.58" rot="R90">
 <attribute name="PROD_ID" value="DIO-09886" x="11.43" y="68.58" size="1.778" layer="27" rot="R90" display="off"/>
@@
 <element name="JP8" library="SparkFun-Connectors" package="1X02" value="M02PTH" x="29.21" y="22.86" smashed="yes" rot="R90"/>
 <element name="JP25" library="SparkFun-Connectors" package="1X02" value="M02PTH" x="31.75" y="41.91" rot="R90"/>
-<element name="R31" library="SparkFun-Resistors" package="0805" value="10K" x="35.56" y="38.1"/>
+<element name="R31" library="SparkFun-Resistors" package="0805" value="10K" x="36.83" y="39.37"/>
 <element name="U$10" library="RitLaunchInitiative" package="TI_CONNECTED_BOOSTER" value="BOOSTER_PACK_CONNECTED" x="31.75" y="34.29" rot="R90"/>
 <element name="JP20" library="SparkFun-Connectors" package="1X03" value="" x="43.815" y="3.81" rot="R90"/>
@@
 <contactref element="U$10" pad="PH0"/>
 <wire x1="40.64" y1="44.45" x2="85.09" y2="54.61" width="0" layer="19" extent="1-1"/>
-<wire x1="38.47" y1="38.1" x2="40.64" y2="44.45" width="0" layer="19" extent="1-1"/>
+<wire x1="39.74" y1="39.37" x2="40.64" y2="44.45" width="0" layer="19" extent="1-1"/>
 </signal>
 <signal name="BATTVOLTAGE">
@@
 <contactref element="R31" pad="1"/>
 <contactref element="U$10" pad="PH1"/>
-<wire x1="34.66" y1="38.1" x2="87.63" y2="54.61" width="0" layer="19" extent="1-1"/>
-<wire x1="31.75" y1="41.91" x2="34.66" y2="38.1" width="0" layer="19" extent="1-1"/>
+<wire x1="35.93" y1="39.37" x2="87.63" y2="54.61" width="0" layer="19" extent="1-1"/>
+<wire x1="31.75" y1="41.91" x2="35.93" y2="39.37" width="0" layer="19" extent="1-1"/>
 </signal>
 <signal name="PSI_3">

Commit message: Finished bulk routing.
Parts:
- removed C16: 10uF, SparkFun-Capacitors:0805
- removed C17: 0.1uf, SparkFun-Capacitors:0805
- removed C18: 100pF, SparkFun-Capacitors:0805
- added R37, R38: 10K, SparkFun-Resistors:0805
- added S2: SWITCH-MOMENTARY-2SMD, SparkFun-Electromechanical:TACTILE-SWITCH-SMD
- moved C14 79.0 mm to (100.3, 39.4)
- moved C15 78.8 mm to (100.3, 37.5)
- moved C13 76.3 mm to (94.0, 41.9), turned to 90 degrees
- moved C10 59.7 mm to (72.4, 31.8), turned to 270 degrees
- moved S1 58.9 mm to (88.9, 64.1), turned to 180 degrees
- moved C8 57.2 mm to (69.8, 35.6), turned to 180 degrees
- moved R32 52.1 mm to (93.3, 60.3), turned to 180 degrees
- moved C2 47.6 mm to (88.3, 76.8), turned to 90 degrees
- moved C19 46.9 mm to (90.2, 76.8), turned to 270 degrees
- moved C1 46.6 mm to (92.1, 76.8)
- moved JP25 11.7 mm to (40.6, 49.5)
- moved JP1777 8.13 mm to (47.0, 49.5), turned to 90 degrees
- moved R31 8.13 mm to (41.9, 45.7), turned to 270 degrees
- moved R30 7.75 mm to (45.1, 45.7), turned to 270 degrees
- moved R34 7.10 mm to (81.9, 77.5), turned to 270 degrees
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Connections:
- new net RST: S2.1, U$10.RST, U$10.RST1
- net +3V3: now also R37.1, R38.1
- net 12V: no longer C16.1, C17.1, C18.1
- net GND: now also S2.3; no longer C16.2, C17.2, C18.2
- net SCL: now also R37.2
- net SDA: now also R38.2
Routing:
- net +3V3: track 138.7 -> 303.9 mm, vias 5 -> 8
- net SCK: track 0.00 -> 143.7 mm, vias 0 -> 11
- net KEYSWITCH_1: track 0.00 -> 57.8 mm, vias 0 -> 2
- net RST: track 0.00 -> 49.2 mm, vias 0 -> 4
- net TILTSWITCH_1: track 0.00 -> 49.1 mm, vias 0 -> 2
- net SW_1: track 0.00 -> 23.7 mm, vias 0 -> 1
- net CS: track 0.00 -> 18.7 mm
- net MISO: track 0.00 -> 17.7 mm
- net FET1: track 29.2 -> 32.2 mm
- net 12V: track 216.7 -> 218.9 mm

Commit message: added alot more ground vias
Routing:
- net CS: track 18.7 -> 27.0 mm, vias 0 -> 2
- net SCK: track 143.7 -> 148.2 mm
