File: Electronics/TestEngine1/InstrumentationBoard.brd (EAGLE design)
At the start: 105.1 x 80 mm, 107 parts, among them IC1 MAX31855, J1 1X2-3.5MM, Q1 MOSFET-NCHANNELBSS123LT1G, Q2 MOSFET-NCHANNELBSS123LT1G, Q3 MOSFET-NCHANNELBSS123LT1G, U1 BMP180

Commit message: minor fixes
Parts:
- moved U$8 27.9 mm to (66.0, 5.08)
Changed lines of the file:
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@@
 <text x="38.735" y="53.975" size="0.8128" layer="21">KeySw</text>
 <text x="45.72" y="53.975" size="0.8128" layer="21">TiltSw</text>
-<text x="92.71" y="45.72" size="3.81" layer="22" rot="MR0">RIT launch Initative</text>
-<text x="92.71" y="41.91" size="2.1844" layer="22" rot="MR0">Instrumentation board</text>
-<text x="54.61" y="41.91" size="2.1844" layer="22" rot="MR0">Rev A</text>
+<text x="72.39" y="44.45" size="3.81" layer="22" rot="MR0">RIT launch Initative</text>
+<text x="72.39" y="40.005" size="2.1844" layer="22" rot="MR0">Instrumentation board</text>
+<text x="72.39" y="36.83" size="2.1844" layer="22" rot="MR0">Rev A</text>
 </plain>
 <attributes>
@@
 <attribute name="PROD_ID" value="SWCH-08247" x="8.89" y="33.655" size="1.778" layer="27" display="off"/>
 </element>
-<element name="U$8" library="RitLaunchInitiative" package="RITLAUNCH_LOGO" value="" x="45.72" y="24.13" rot="MR0"/>
+<element name="U$8" library="RitLaunchInitiative" package="RITLAUNCH_LOGO" value="" x="66.04" y="5.08" rot="MR0"/>
 </elements>
 <signals>

Commit message: changed some minor component values and added part numbers
added attributes to parts for digikey part numbers and changed some
values to match whats available on the market
Parts:
- R14, R16, R18: value 1.7k -> 1.8k
- R19: value 9k -> 3k
- R20: value 3k -> 1k
- R21: value 100 -> 226
- R22: value 220 -> 560
- R23: value 680 -> 2k
Changed lines of the file:
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@@
 <element name="C1" library="SparkFun-Capacitors" package="0805" value="10uF" x="92.075" y="76.835" rot="R90"/>
 <element name="C2" library="SparkFun-Capacitors" package="0805" value="10uF" x="88.265" y="76.835" rot="R90"/>
-<element name="C3" library="microbuilder" package="_0805" value="0.01µF" x="95.25" y="72.39" rot="R270"/>
+<element name="C3" library="microbuilder" package="_0805" value="0.01µF" x="95.25" y="72.39" rot="R270">
+<attribute name="DIGIKEY" value="490-1664-1-ND" x="95.25" y="72.39" size="1.778" layer="27" rot="R270" display="off"/>
+</element>
 <element name="FB1" library="microbuilder" package="_0805" value="Ferrite" x="96.52" y="78.105" smashed="yes" rot="R180">
 <attribute name="NAME" x="98.1075" y="76.835" size="0.8128" layer="25" ratio="18" rot="R180"/>
+<attribute name="DIGIKEY" value="732-1609-1-ND" x="96.52" y="78.105" size="1.778" layer="27" rot="R180" display="off"/>
 </element>
 <element name="FB2" library="microbuilder" package="_0805" value="Ferrite" x="96.52" y="66.675" smashed="yes" rot="R180">
 <attribute name="NAME" x="98.1075" y="65.405" size="0.8128" layer="25" ratio="18" rot="R180"/>
+<attribute name="DIGIKEY" value="732-1609-1-ND" x="96.52" y="66.675" size="1.778" layer="27" rot="R180" display="off"/>
 </element>
 <element name="IC1" library="adafruit" package="SO08" value="MAX31855" x="88.9" y="72.39" smashed="yes" rot="R90"/>
@@
 <attribute name="DIGIKEY_PART_NUMBER" value="INA125UA-ND" x="57.15" y="12.065" size="1.778" layer="27" display="off"/>
 </element>
-<element name="U$2" library="RitLaunchInitiative" package="TO-252" value="MC33269DTRK" x="93.98" y="33.02" smashed="yes" rot="R90"/>
+<element name="U$2" library="RitLaunchInitiative" package="TO-252" value="MC33269DTRK" x="93.98" y="33.02" smashed="yes" rot="R90">
+<attribute name="DIGIKEY" value="MC33269DTRK-5.0GOSCT-ND" x="93.98" y="33.02" size="1.778" layer="27" rot="R90" display="off"/>
+</element>
 <element name="U$3" library="RitLaunchInitiative" package="SOT223" value="TC1262" x="82.55" y="33.02" smashed="yes" rot="R90">
 <attribute name="VALUE" x="82.7405" y="31.9405" size="0.4064" layer="27" rot="R90"/>
+<attribute name="DIGIKEY" value="TC1262-3.3VDBCT-ND" x="82.55" y="33.02" size="1.778" layer="27" rot="R90" display="off"/>
 </element>
 <element name="C4" library="SparkFun-Capacitors" package="0805" value="0.33uF" x="100.965" y="33.02" rot="R270"/>
@@
 <attribute name="VALUE" x="44.45" y="2.54" size="1.27" layer="27" rot="R90"/>
 </element>
-<element name="R14" library="SparkFun-Resistors" package="0805" value="1.7k" x="41.275" y="12.065" rot="R270"/>
-<element name="R15" library="SparkFun-Resistors" package="0805" value="3.3k" x="41.275" y="15.875" rot="R270"/>
+<element name="R14" library="SparkFun-Resistors" package="0805" value="1.8k" x="41.275" y="12.065" rot="R270">
+<attribute name="DIGIKEY" value="RMCF0805FT1K80CT-ND" x="41.275" y="12.065" size="1.778" layer="27" rot="R270" display="off"/>
+</element>
+<element name="R15" library="SparkFun-Resistors" package="0805" value="3.3k" x="41.275" y="15.875" rot="R270">
+<attribute name="DIGIKEY" value="RHM3.30KCHCT-ND" x="41.275" y="15.875" size="1.778" layer="27" rot="R270" display="off"/>
+</element>
 <element name="U1" library="SparkFun-Sensors" package="BMP180" value="BMP180" x="69.215" y="31.75" smashed="yes" rot="R270">
 <attribute name="NAME" x="67.85" y="28.035" size="1.27" layer="25"/>
@@
 <attribute name="VALUE" x="8.255" y="48.26" size="1.27" layer="27" rot="R270"/>
 </element>
-<element name="LED1" library="adafruit" package="RGBLED5050" value="RGBLED5050" x="73.66" y="72.39" smashed="yes" rot="R270"/>
+<element name="LED1" library="adafruit" package="RGBLED5050" value="RGBLED5050" x="73.66" y="72.39" smashed="yes" rot="R270">
+<attribute name="DIGIKEY" value="1516-1131-1-ND" x="73.66" y="72.39" size="1.778" layer="27" rot="R270" display="off"/>
+</element>
 <element name="JP1777" library="SparkFun-Connectors" package="1X02" value="M02PTH" x="46.99" y="49.53" smashed="yes" rot="R90"/>
 <element name="S1" library="SparkFun-Electromechanical" package="TACTILE-SWITCH-SMD" value="SWITCH-MOMENTARY-2SMD" x="88.9" y="64.135" smashed="yes" rot="R180">
@@
 <attribute name="DIGIKEY" value="SS110-TPCT-ND" x="49.53" y="68.58" size="1.778" layer="27" rot="R90" display="off"/>
 </element>
-<element name="R19" library="SparkFun-Resistors" package="0805" value="9k" x="97.155" y="38.1" rot="R180"/>
-<element name="R20" library="SparkFun-Resistors" package="0805" value="3k" x="92.075" y="38.1" rot="R180"/>
+<element name="R19" library="SparkFun-Resistors" package="0805" value="3k" x="97.155" y="38.1" rot="R180"/>
+<element name="R20" library="SparkFun-Resistors" package="0805" value="1k" x="92.075" y="38.1" rot="R180"/>
 <element name="R5" library="SparkFun-Resistors" package="0805" value="10k" x="21.59" y="19.05" rot="R90"/>
 <element name="JP5" library="SparkFun-Connectors" package="1X02" value="M02PTH" x="21.59" y="22.86" smashed="yes" rot="R90"/>
@@
 <attribute name="VALUE" x="41.91" y="2.54" size="1.27" layer="27" rot="R90"/>
 </element>
-<element name="R16" library="SparkFun-Resistors" package="0805" value="1.7k" x="38.735" y="12.065" rot="R270"/>
-<element name="R17" library="SparkFun-Resistors" package="0805" value="3.3k" x="36.195" y="12.065" rot="R90"/>
+<element name="R16" library="SparkFun-Resistors" package="0805" value="1.8k" x="38.735" y="12.065" rot="R270">
+<attribute name="DIGIKEY" value="RMCF0805FT1K80CT-ND" x="38.735" y="12.065" size="1.778" layer="27" rot="R270" display="off"/>
+</element>
+<element name="R17" library="SparkFun-Resistors" package="0805" value="3.3k" x="36.195" y="12.065" rot="R90">
+<attribute name="DIGIKEY" value="RHM3.30KCHCT-ND" x="36.195" y="12.065" size="1.778" layer="27" rot="R90" display="off"/>
+</element>
 <element name="JP19" library="SparkFun-Connectors" package="1X03" value="" x="13.97" y="46.99" smashed="yes" rot="R270">
 <attribute name="VALUE" x="10.795" y="48.26" size="1.27" layer="27" rot="R270"/>
@@
 <element name="C19" library="SparkFun-Capacitors" package="0805" value="0.1uf" x="90.17" y="76.835" rot="R270"/>
 <element name="D9" library="SparkFun-LED" package="LED-1206" value="" x="91.44" y="45.72" rot="R90">
-<attribute name="DIGIKEY" value="350-2048-1-ND" x="91.44" y="45.72" size="1.778" layer="27" rot="R90" display="off"/>
-</element>
-<element name="R21" library="SparkFun-Resistors" package="0805" value="100" x="86.36" y="41.275" rot="R90"/>
-<element name="R22" library="SparkFun-Resistors" package="0805" value="220" x="88.9" y="41.275" rot="R90"/>
-<element name="R23" library="SparkFun-Resistors" package="0805" value="680" x="91.44" y="41.275" rot="R90"/>
+<attribute name="DIGIKEY" value="160-1405-1-ND" x="91.44" y="45.72" size="1.778" layer="27" rot="R90" display="off"/>
+</element>
+<element name="R21" library="SparkFun-Resistors" package="0805" value="226" x="86.36" y="41.275" rot="R90">
+<attribute name="DIGIKEY" value="P226CCT-ND" x="86.36" y="41.275" size="1.778" layer="27" rot="R90" display="off"/>
+</element>
+<element name="R22" library="SparkFun-Resistors" package="0805" value="560" x="88.9" y="41.275" rot="R90">
+<attribute name="DIGIKEY" value="P560CCT-ND" x="88.9" y="41.275" size="1.778" layer="27" rot="R90" display="off"/>
+</element>
+<element name="R23" library="SparkFun-Resistors" package="0805" value="2k" x="91.44" y="41.275" rot="R90">
+<attribute name="DIGIKEY" value="P2.00KCCT-ND" x="91.44" y="41.275" size="1.778" layer="27" rot="R90" display="off"/>
+</element>
 <element name="D7" library="SparkFun-LED" package="LED-1206" value="" x="88.9" y="45.72" rot="R90">
-<attribute name="DIGIKEY" value="350-2048-1-ND" x="88.9" y="45.72" size="1.778" layer="27" rot="R90" display="off"/>
+<attribute name="DIGIKEY" value="160-1405-1-ND" x="88.9" y="45.72" size="1.778" layer="27" rot="R90" display="off"/>
 </element>
 <element name="D8" library="SparkFun-LED" package="LED-1206" value="" x="86.36" y="45.72" rot="R90">
-<attribute name="DIGIKEY" value="350-2048-1-ND" x="86.36" y="45.72" size="1.778" layer="27" rot="R90" display="off"/>
+<attribute name="DIGIKEY" value="160-1405-1-ND" x="86.36" y="45.72" size="1.778" layer="27" rot="R90" display="off"/>
 </element>
 <element name="U$9" library="RitLaunchInitiative" package="TO-252" value="FDD3706" x="30.48" y="67.31" smashed="yes">
@@
 <attribute name="VALUE" x="46.99" y="2.54" size="1.27" layer="27" rot="R90"/>
 </element>
-<element name="R18" library="SparkFun-Resistors" package="0805" value="1.7k" x="43.815" y="12.065" rot="R270"/>
-<element name="R36" library="SparkFun-Resistors" package="0805" value="3.3k" x="45.72" y="12.065" rot="R90"/>
+<element name="R18" library="SparkFun-Resistors" package="0805" value="1.8k" x="43.815" y="12.065" rot="R270">
+<attribute name="DIGIKEY" value="RMCF0805FT1K80CT-ND" x="43.815" y="12.065" size="1.778" layer="27" rot="R270" display="off"/>
+</element>
+<element name="R36" library="SparkFun-Resistors" package="0805" value="3.3k" x="45.72" y="12.065" rot="R90">
+<attribute name="DIGIKEY" value="RHM3.30KCHCT-ND" x="45.72" y="12.065" size="1.778" layer="27" rot="R90" display="off"/>
+</element>
 <element name="R37" library="SparkFun-Resistors" package="0805" value="10K" x="42.545" y="26.035" rot="R90"/>
 <element name="R38" library="SparkFun-Resistors" package="0805" value="10K" x="42.545" y="29.845" rot="R270"/>
