File: MITAvionics/MITAvionicsRevA.sch (EAGLE design)
At the start: 50 parts, among them IC1 4050D, IC2 4050D, IC3 4050D, Q1 MOSFET-NCHANNELBSS123LT1G, Q2 MOSFET-NCHANNELBSS123LT1G, Q3 MOSFET-NCHANNELBSS123LT1G, Q4 MOSFET-NCHANNELBSS123LT1G, U1 ARDUINO-MEGAFULL, X1 MICROSD

Commit message: Work in progress
Parts:
- added C9: 10uF, SparkFun-Capacitors:CAP0805
- added D5, D6: (no value), SparkFun-LED:LED1206
- added JP1, JP2: (no value), SparkFun-Connectors:M023.5MM
- added JP3, JP4, JP5: (no value), SparkFun-Connectors:M03PTH
- added JP6: (no value), SparkFun-Connectors:M06SMD-1MM
- added Q5, Q6, Q7, Q8, Q9: MOSFET-NCHANNELBSS123LT1G, SparkFun-DiscreteSemi:MOSFET-NCHANNELBSS123LT1G
- added R10, R12, R26, R27, R28, R7: 10K, SparkFun-Resistors:RESISTOR0805-RES
- added R11, R15, R16, R29, R30, R9: 1k, SparkFun-Resistors:RESISTOR0805-RES
- added R13, R14: 10k, SparkFun-Resistors:RESISTOR0805-RES
- added R17, R25: 0, SparkFun-Resistors:RESISTOR0805-RES
- added R18: 40, SparkFun-Resistors:RESISTOR0805-RES
- added SJ2: JUMPER-PAD-2-NC_BY_TRACE, SparkFun-Passives:JUMPER-PAD-2-NC_BY_TRACE
- added SJ6: JUMPER-PAD-3-2OF3_NC_BY_TRACE_SMALL, SparkFun-Passives:JUMPER-PAD-3-2OF3_NC_BY_TRACE_SMALL
- added U$4: FDD3706, RitLaunchInitiative:FDD3706
- added U$5: LTST-C19FD1WT, RitLaunchInitiative:LTST-C19FD1WT
- added U$6: JST_VERTICAL, SparkFun-Connectors:JST_VERTICAL
Connections:
- new net BUZZER: Q4.G, R6.1
- new net FET1: R12.1, U$4.G
- new net GPS_BACKUP_V: U$6.5
- new net GPS_CTL: U$6.6
- new net GPS_RX: U$6.4
- new net GPS_TX: U$6.3
- new net G_RDY: JP6.4
- new net HOTWIRE_CONTINUITY: R13.2, R14.1
- new net L_RDY: JP6.5
- new net N$17: D5.A, R9.2
- new net N$18: D5.C, Q5.D
- new net N$19: D6.A, R11.2
- new net N$20: D6.C, Q6.D
- new net N$21: Q9.D, R17.2
- new net N$22: Q7.D, R18.2
- new net N$26: Q8.D, R25.2
- new net N$27: JP1.1, R15.1
- new net N$28: R29.1, R30.1, SJ6.2
- new net N$30: R16.1, SJ2.1
- new net N$36: R17.1, U$5.GREEN
- new net N$37: R18.1, U$5.RED
- new net N$38: R25.1, U$5.BLUE
- new net PYRO_MONITOR: R15.2, SJ2.2
- new net SERVO_1: JP3.3, JP4.3, JP5.3
- new net STATUS_LED_1: Q5.G, R7.1
- new net STATUS_LED_2: Q6.G, R10.1
- new net STATUS_LED_BLUE: Q8.G, R28.1
- new net STATUS_LED_GREEN: Q9.G, R26.1
- new net STATUS_LED_RED: Q7.G, R27.1
- net +3V3: now also C9.1, JP6.1, R11.1, R9.1, SJ6.1, U$5.VCC, U$6.2
- net 12V: no longer C13.1, C14.1, C15.1
- net 5V: now also SJ6.3
- net GND: now also C9.2, JP1.2, JP3.1, JP4.1, JP5.1, JP6.6, Q5.S, Q6.S, Q7.S, Q8.S, Q9.S, R10.2, R12.2, R14.2, R16.2, R26.2, R27.2, R28.2, R7.2, U$4.S, U$6.1
- net N$5: now also JP2.1, R13.1, U$4.D; no longer SJ4.1
- net RESET: now also SJ4.1
- net SCL: now also JP6.3, R29.2
- net SDA: now also JP6.2, R30.2
- net V_BATT: now also C13.1, C14.1, C15.1, JP2.2, JP3.2, JP4.2, JP5.2
Other:
- note added: "7Volts"
- note added: "Altimeter ground"
- moved on the sheet: C1, IC1P, Q3, R24, SJ4

Commit message: Finished Schematic started routing
Parts:
- removed IC2, IC3: 4050D, 40xx:4050D
- removed J2, J3: (no value), SparkFun-Connectors:BANANA_CONN
- removed U$6: JST_VERTICAL, SparkFun-Connectors:JST_VERTICAL
- added GPS_HEADER: JST_VERTICAL, SparkFun-Connectors:JST_VERTICAL
- added IMU_HEADER: (no value), SparkFun-Connectors:M06SMD-1MM
- added JP7, JP8, JP9: (no value), SparkFun-Connectors:M024UCON-15767
- added R31: 10K, SparkFun-Resistors:RESISTOR0805-RES
- added SJ7, SJ8: JUMPER-PAD-2-NC_BY_TRACE, SparkFun-Passives:JUMPER-PAD-2-NC_BY_TRACE
- JP6: device SparkFun-Connectors:M06SMD-1MM -> SparkFun-Connectors:M023.5MM; DIGIKEY 455-1806-2-ND -> (none)
Connections:
- net N$3 renamed XBEE_RX
- removed net FET1: R12.1, U$4.G
- removed net GPS_BACKUP_V: U$6.5
- removed net GPS_CTL: U$6.6
- removed net RX0_MEGA: Q2.G, R4.1, U$1.DOUT, U1.0(RX0)
- removed net RX1_MEGA: U1.19(RX1)
- removed net RX2_MEGA: U1.17(RX2)
- removed net RX3_MEGA: U1.15(RX3)
- removed net TX0_MEGA: IC1A.I, Q1.G, R2.1, U1.1(TX0)
- removed net TX1_MEGA: U1.18(TX1)
- removed net TX2_MEGA: U1.16(TX2)
- removed net TX3_MEGA: U1.14(TX3)
- new net ARM_SWITCH: JP9.2, R31.1, U1.30
- new net GPS_STATUS: GPS_HEADER.6, U1.22
- new net HOTWIRE_FET: R12.1, U$4.G, U1.10
- new net N$29: SJ7.1, U1.VIN
- new net N$3: SJ8.1, U1.3.3V
- new net SERVO_2: JP4.3, U1.12
- new net SERVO_3: JP5.3, U1.13
- new net XBEE_RX_5V: IC1A.I, R4.1, U1.1(TX0)
- new net XBEE_TX: R2.1, U$1.DOUT, U1.0(RX0)
- net +3V3: now also B1.2, IMU_HEADER.6, JP7.2, JP9.1, SJ8.2; no longer IC2P.VDD, IC3P.VDD, JP6.1, U$6.2
- net 5V: now also GPS_HEADER.2
- net BATTVOLTAGE: now also U1.A4
- net BUZZER: now also U1.42
- net CLK: now also U1.52
- net CS: now also U1.53
- net DI: now also U1.51
- net DO: now also U1.50
- net GND: now also GPS_HEADER.1, GPS_HEADER.5, IMU_HEADER.1, JP1.1, JP6.1, R31.2, U1.GND@0, U1.GND@1, U1.GND@2, U1.GND@3, U1.GND@4; no longer IC2P.VSS, IC3P.VSS, J3.1, JP1.2, JP6.6, U$6.1
- net GPS_RX: now also GPS_HEADER.3, U1.18(TX1); no longer U$6.4
- net GPS_TX: now also GPS_HEADER.4, U1.19(RX1); no longer U$6.3
- net G_RDY: now also IMU_HEADER.4, U1.34; no longer JP6.4
- net HOTWIRE_CONTINUITY: now also U1.A6
- net L_RDY: now also IMU_HEADER.5, U1.32; no longer JP6.5
- net N$27: now also JP1.2; no longer JP1.1
- net N$5: now also JP2.2; no longer JP2.1
- net N$8: now also B1.1, JP7.1
- net PYRO_MONITOR: now also U1.A5
- net SCL: now also IMU_HEADER.3; no longer JP6.3
- net SDA: now also IMU_HEADER.2; no longer JP6.2
- net SERVO_1: now also U1.11; no longer JP4.3, JP5.3
- net STATUS_LED_1: now also U1.44
- net STATUS_LED_2: now also U1.46
- net STATUS_LED_BLUE: now also U1.40
- net STATUS_LED_GREEN: now also U1.36
- net STATUS_LED_RED: now also U1.38
- net V_BATT: now also JP2.1, JP6.2, SJ7.2; no longer J2.1, JP2.2
Other:
- note added: "10-DOF IMU header"
- note added: "DataLogging"
- note added: "GPS HEADER EM-506"
- note added: "Navigation"
- note added: "Normally Closed"
- note added: "Over air Re-programming"
- note added: "Remove Before Launch / ARM button"
- note added: "Select between 3v3 / 5v I2C Bus"
- moved on the sheet: B1, C1, C9, D4, D5, D6, IC1B, IC1C, IC1D, IC1E, IC1F, JP1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

Commit message: Routing Complete
Parts:
- removed D4, D5, D6: (no value), SparkFun-LED:LED1206
- removed IC1: 4050D, 40xx:4050D
- removed JP7, JP8, JP9: (no value), SparkFun-Connectors:M024UCON-15767
- removed Q5, Q6: MOSFET-NCHANNELBSS123LT1G, SparkFun-DiscreteSemi:MOSFET-NCHANNELBSS123LT1G
- removed R10, R31, R7: 10K, SparkFun-Resistors:RESISTOR0805-RES
- removed R11, R8, R9: 1k, SparkFun-Resistors:RESISTOR0805-RES
- removed X1: MICROSD, adafruit:MICROSD
- added C10, C11, C12: 0.1uf, SparkFun-Capacitors:CAP0805
- added SJ10, SJ9: JUMPER-PAD-2-NC_BY_TRACE, SparkFun-Passives:JUMPER-PAD-2-NC_BY_TRACE
- added U2, U3: (no value), SparkFun-DigitalIC:TXB0104PWRSOIC14
- added U4: USD-SOCKET, SparkFun-Connectors:USD-SOCKET
- C9: value 10uF -> 0.1uf; DIGIKEY 490-3886-1-ND -> (none)
- R23: value 2k -> 1k
Connections:
- removed net 12V: R23.1
- removed net ARM_SWITCH: JP9.2, R31.1, U1.30
- removed net CD: X1.CARD_DETECT
- removed net N$12: D3.C, Q2.D
- removed net N$13: IC1D.O, X1.SCLK
- removed net N$14: IC1E.O, R8.2, X1.CS
- removed net N$16: IC1C.O, X1.DATA_IN
- removed net N$18: D5.C, Q5.D
- removed net N$19: D6.A, R11.2
- removed net N$20: D6.C, Q6.D
- removed net STATUS_LED_1: Q5.G, R7.1, U1.44
- removed net STATUS_LED_2: Q6.G, R10.1, U1.46
- removed net XBEE_RX: IC1A.O, U$1.DIN
- removed net XBEE_TX: R2.1, U$1.DOUT, U1.0(RX0)
- new net SD_CS: U2.A3, U4.CS
- new net SD_DI: U2.A4, U4.DI
- new net SD_DO: U2.A1, U4.DO
- new net SD_SCK: U2.A2, U4.SCK
- new net XBEE_RX_3V3: U$1.DIN, U3.A1
- new net XBEE_TX_3V3: U$1.DOUT, U3.A2
- new net XBEE_TX_5V: Q1.G, R2.1, U1.0(RX0), U3.B2
- net +3V3: now also C11.1, D2.A, D3.A, IMU_HEADER.1, SJ10.2, SJ9.2, U2.VCCA, U3.VCCA, U4.VCC; no longer IC1P.VDD, IMU_HEADER.6, JP7.2, JP9.1, R11.1, R3.1, R5.1, R9.1, X1.VDD
- net 5V: now also C10.1, C12.1, U2.VCCB, U3.VCCB
- net BATTVOLTAGE: now also U1.A0(RX0); no longer U1.A4
- net BUZZER: now also U1.36; no longer U1.42
- net CLK: now also U2.B2; no longer IC1D.I, IC1F.I
- net CS: now also U2.B3; no longer IC1E.I
- net DI: now also U2.B4; no longer IC1C.I
- net DO: now also U2.B1; no longer X1.DATA_OUT
- net GND: now also C10.2, C11.2, C12.2, IMU_HEADER.6, JP1.2, U2.GND, U3.GND, U4.CD1, U4.CD2, U4.GND, U4.SHIELD@1, U4.SHIELD@3; no longer IC1P.VSS, IMU_HEADER.1, JP1.1, Q5.S, Q6.S, R10.2, R31.2, R7.2, X1.GND, X1.GND1, X1.VSS
- net G_RDY: now also IMU_HEADER.5, U1.28; no longer IMU_HEADER.4, U1.34
- net HOTWIRE_CONTINUITY: now also U1.A1(TX0); no longer U1.A6
- net L_RDY: now also IMU_HEADER.4, U1.26; no longer IMU_HEADER.5, U1.32
- net N$10: now also R3.1; no longer Q1.D
- net N$11: now also Q1.D, R3.2; no longer D3.A, R5.2
- net N$15: now also SJ9.1, U2.OE; no longer D4.C, R8.1
- net N$17: now also SJ10.1, U3.OE; no longer D5.A, R9.2
- net N$2: now also U3.A3; no longer IC1B.I
- net N$27: now also JP1.1; no longer JP1.2
- net N$4: now also D3.C, R5.1; no longer D4.A, IC1F.O
- net N$8: no longer JP7.1
- net N$9: now also Q2.D, R5.2; no longer D2.A, R3.2
- net PYRO_MONITOR: now also U1.A2; no longer U1.A5
- net RST_CTL: now also U1.9, U3.B3; no longer IC1B.O
- net STATUS_LED_BLUE: now also U1.34; no longer U1.40
- net STATUS_LED_GREEN: now also U1.30; no longer U1.36
- net STATUS_LED_RED: now also U1.32; no longer U1.38
- net V_BATT: now also R23.1
- net XBEE_RX_5V: now also Q2.G, U3.B1; no longer IC1A.I
Other:
- note added: "might need to replace with 226 value"
- note removed: "Normally Closed"
- note removed: "Remove Before Launch / ARM button"
- moved on the sheet: C2, C3, C8, C9, D1, D2, D3, JP1, JP2, Q1, Q2, R1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

Commit message: moved small things around added silk screen
Parts:
- added JP7: (no value), SparkFun-Connectors:M02PTH
Changed lines of the file:
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@@
 <part name="GND32" library="supply1" deviceset="GND" device=""/>
 <part name="+3V16" library="supply1" deviceset="+3V3" device=""/>
+<part name="JP7" library="SparkFun-Connectors" deviceset="M02" device="PTH"/>
 </parts>
 <sheets>
@@
 <instance part="GND32" gate="1" x="434.34" y="22.86"/>
 <instance part="+3V16" gate="G$1" x="431.8" y="71.12"/>
+<instance part="JP7" gate="G$1" x="-30.48" y="10.16"/>
 </instances>
 <busses>
