File: MITAvionics/MITAvionicsRevA.brd (EAGLE design)
At the start: 100 x 80 mm, 50 parts, among them IC1 4050D, IC2 4050D, IC3 4050D, Q1 MOSFET-NCHANNELBSS123LT1G, Q2 MOSFET-NCHANNELBSS123LT1G, Q3 MOSFET-NCHANNELBSS123LT1G, Q4 MOSFET-NCHANNELBSS123LT1G, U1 ARDUINO-MEGAFULL, X1 MICROSD

Commit message: Work in progress
Parts:
- added C9: 10uF, SparkFun-Capacitors:0805
- added D5, D6: (no value), SparkFun-LED:LED-1206
- added JP1, JP2: (no value), SparkFun-Connectors:SCREWTERMINAL-3.5MM-2
- added JP3, JP4, JP5: (no value), SparkFun-Connectors:1X03
- added JP6: (no value), SparkFun-Connectors:1X06-1MM
- added Q5, Q6, Q7, Q8, Q9: MOSFET-NCHANNELBSS123LT1G, SparkFun-DiscreteSemi:SOT23-3
- added R10, R12, R26, R27, R28, R7: 10K, SparkFun-Resistors:0805
- added R11, R15, R16, R29, R30, R9: 1k, SparkFun-Resistors:0805
- added R13, R14: 10k, SparkFun-Resistors:0805
- added R17, R25: 0, SparkFun-Resistors:0805
- added R18: 40, SparkFun-Resistors:0805
- added SJ2: JUMPER-PAD-2-NC_BY_TRACE, SparkFun-Passives:PAD-JUMPER-2-NC_BY_TRACE_YES_SILK
- added SJ6: JUMPER-PAD-3-2OF3_NC_BY_TRACE_SMALL, SparkFun-Passives:PAD-JUMPER-3-2OF3_NC_BY_TRACE_YES_SILK_FULL_BOX
- added U$4: FDD3706, RitLaunchInitiative:TO-252
- added U$5: LTST-C19FD1WT, RitLaunchInitiative:SMD-4
- added U$6: JST_VERTICAL, SparkFun-Connectors:JST-6-SMD-VERT-1.0MM
Connections:
- new net BUZZER: Q4.1, R6.1
- new net FET1: R12.1, U$4.1
- new net GPS_BACKUP_V: U$6.5
- new net GPS_CTL: U$6.6
- new net GPS_RX: U$6.4
- new net GPS_TX: U$6.3
- new net G_RDY: JP6.4
- new net HOTWIRE_CONTINUITY: R13.2, R14.1
- new net L_RDY: JP6.5
- new net N$17: D5.A, R9.2
- new net N$18: D5.C, Q5.3
- new net N$19: D6.A, R11.2
- new net N$20: D6.C, Q6.3
- new net N$21: Q9.3, R17.2
- new net N$22: Q7.3, R18.2
- new net N$26: Q8.3, R25.2
- new net N$27: JP1.1, R15.1
- new net N$28: R29.1, R30.1, SJ6.2
- new net N$30: R16.1, SJ2.1
- new net N$36: R17.1, U$5.P$3
- new net N$37: R18.1, U$5.P$2
- new net N$38: R25.1, U$5.P$1
- new net PYRO_MONITOR: R15.2, SJ2.2
- new net SERVO_1: JP3.3, JP4.3, JP5.3
- new net STATUS_LED_1: Q5.1, R7.1
- new net STATUS_LED_2: Q6.1, R10.1
- new net STATUS_LED_BLUE: Q8.1, R28.1
- new net STATUS_LED_GREEN: Q9.1, R26.1
- new net STATUS_LED_RED: Q7.1, R27.1
- net +3V3: now also C9.1, JP6.1, R11.1, R9.1, SJ6.1, U$5.P$4, U$6.2
- net 12V: no longer C13.1, C14.1, C15.1
- net 5V: now also SJ6.3
- net GND: now also C9.2, JP1.2, JP3.1, JP4.1, JP5.1, JP6.6, Q5.2, Q6.2, Q7.2, Q8.2, Q9.2, R10.2, R12.2, R14.2, R16.2, R26.2, R27.2, R28.2, R7.2, U$4.3, U$6.1
- net N$5: now also JP2.1, R13.1, U$4.2; no longer SJ4.1
- net RESET: now also SJ4.1
- net SCL: now also JP6.3, R29.2
- net SDA: now also JP6.2, R30.2
- net V_BATT: now also C13.1, C14.1, C15.1, JP2.2, JP3.2, JP4.2, JP5.2

Commit message: Finished Schematic started routing
Parts:
- removed IC2, IC3: 4050D, 40xx:SO16
- removed J2, J3: (no value), SparkFun-Connectors:BANANA_CONN
- removed U$6: JST_VERTICAL, SparkFun-Connectors:JST-6-SMD-VERT-1.0MM
- added GPS_HEADER: JST_VERTICAL, SparkFun-Connectors:JST-6-SMD-VERT-1.0MM
- added IMU_HEADER: (no value), SparkFun-Connectors:1X06-1MM
- added JP7, JP8, JP9: (no value), SparkFun-Connectors:JST-2-SMD-VERT
- added R31: 10K, SparkFun-Resistors:0805
- added SJ7, SJ8: JUMPER-PAD-2-NC_BY_TRACE, SparkFun-Passives:PAD-JUMPER-2-NC_BY_TRACE_YES_SILK
- JP6: device SparkFun-Connectors:1X06-1MM -> SparkFun-Connectors:SCREWTERMINAL-3.5MM-2
- moved JP6 351.4 mm to (45.7, 14.0)
- moved U$5 325.3 mm to (36.8, 33.0)
- moved JP1 319.5 mm to (71.1, 12.7)
- moved SJ2 316.5 mm to (66.0, 7.62), flipped to the bottom
- moved JP5 313.4 mm to (1.91, 3.17), turned to 90 degrees
- moved R16 310.5 mm to (66.7, 10.2), turned to 90 degrees
- moved JP4 310.4 mm to (4.45, 3.17), turned to 90 degrees
- moved JP3 307.4 mm to (6.99, 3.17), turned to 90 degrees
- moved R15 307.1 mm to (64.8, 10.2), turned to 270 degrees
- moved R14 283.4 mm to (29.2, 22.9), turned to 90 degrees
- moved R13 279.1 mm to (26.7, 21.6), turned to 90 degrees
- moved JP2 276.4 mm to (24.1, 4.45)
- moved R12 268.4 mm to (19.7, 19.1), turned to 180 degrees
- moved U$4 252.9 mm to (21.6, 14.6), turned to 270 degrees
- moved X1 216.1 mm to (16.5, 45.1), turned to 270 degrees
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Connections:
- net N$3 renamed XBEE_RX
- removed net FET1: R12.1, U$4.1
- removed net GPS_BACKUP_V: U$6.5
- removed net GPS_CTL: U$6.6
- removed net RX0_MEGA: Q2.1, R4.1, U$1.2, U1.0
- removed net RX1_MEGA: U1.19
- removed net RX2_MEGA: U1.17
- removed net RX3_MEGA: U1.15
- removed net TX0_MEGA: IC1.3, Q1.1, R2.1, U1.1
- removed net TX1_MEGA: U1.18
- removed net TX2_MEGA: U1.16
- removed net TX3_MEGA: U1.14
- new net ARM_SWITCH: JP9.VCC, R31.1, U1.30
- new net GPS_STATUS: GPS_HEADER.6, U1.22
- new net HOTWIRE_FET: R12.1, U$4.1, U1.10
- new net N$29: SJ7.1, U1.VIN
- new net N$3: SJ8.1, U1.3.3V
- new net SERVO_2: JP4.3, U1.12
- new net SERVO_3: JP5.3, U1.13
- new net XBEE_RX_5V: IC1.3, R4.1, U1.1
- new net XBEE_TX: R2.1, U$1.2, U1.0
- net +3V3: now also B1.-, IMU_HEADER.6, JP7.VCC, JP9.GND, SJ8.2; no longer IC2.1, IC3.1, JP6.1, U$6.2
- net 5V: now also GPS_HEADER.2
- net BATTVOLTAGE: now also U1.A4
- net BUZZER: now also U1.42
- net CLK: now also U1.52
- net CS: now also U1.53
- net DI: now also U1.51
- net DO: now also U1.50
- net GND: now also GPS_HEADER.1, GPS_HEADER.5, IMU_HEADER.1, JP1.1, JP6.1, R31.2, U1.GND@0, U1.GND@1, U1.GND@2, U1.GND@3, U1.GND@4; no longer IC2.8, IC3.8, J3.P$1, JP1.2, JP6.6, U$6.1
- net GPS_RX: now also GPS_HEADER.3, U1.18; no longer U$6.4
- net GPS_TX: now also GPS_HEADER.4, U1.19; no longer U$6.3
- net G_RDY: now also IMU_HEADER.4, U1.34; no longer JP6.4
- net HOTWIRE_CONTINUITY: now also U1.A6
- net L_RDY: now also IMU_HEADER.5, U1.32; no longer JP6.5
- net N$27: now also JP1.2; no longer JP1.1
- net N$5: now also JP2.2; no longer JP2.1
- net N$8: now also B1.+, JP7.GND
- net PYRO_MONITOR: now also U1.A5
- net SCL: now also IMU_HEADER.3; no longer JP6.3
- net SDA: now also IMU_HEADER.2; no longer JP6.2
- net SERVO_1: now also U1.11; no longer JP4.3, JP5.3
- net STATUS_LED_1: now also U1.44
- net STATUS_LED_2: now also U1.46
- net STATUS_LED_BLUE: now also U1.40
- net STATUS_LED_GREEN: now also U1.36
- net STATUS_LED_RED: now also U1.38
- net V_BATT: now also JP2.1, JP6.2, SJ7.2; no longer J2.P$1, JP2.2
Routing:
- net HOTWIRE_FET: track 0.00 -> 79.0 mm, vias 0 -> 1
- net SERVO_1: track 0.00 -> 70.9 mm
- net SERVO_2: track 0.00 -> 69.5 mm
- net SERVO_3: track 0.00 -> 69.2 mm
- net V_BATT: track 0.00 -> 64.8 mm
- net 5V: track 0.00 -> 23.0 mm
- net N$5: track 0.00 -> 15.8 mm, vias 0 -> 3
- net GND: track 0.00 -> 10.2 mm, vias 0 -> 53
- net RESET: track 0.00 -> 8.41 mm
- net +3V3: track 0.00 -> 6.37 mm, vias 0 -> 1
- net N$38: track 0.00 -> 5.89 mm
- net N$29: track 0.00 -> 3.57 mm
- net N$3: track 0.00 -> 2.67 mm
- added copper zone on layer 1, net GND
- added copper zone on layer 16, net GND
Other:
- board size 100 x 80 mm -> 101.6 x 53.3 mm

Commit message: Routing Complete
Parts:
- removed D4, D5, D6: (no value), SparkFun-LED:LED-1206
- removed IC1: 4050D, 40xx:SO16
- removed JP7, JP8, JP9: (no value), SparkFun-Connectors:JST-2-SMD-VERT
- removed Q5, Q6: MOSFET-NCHANNELBSS123LT1G, SparkFun-DiscreteSemi:SOT23-3
- removed R10, R31, R7: 10K, SparkFun-Resistors:0805
- removed R11, R8, R9: 1k, SparkFun-Resistors:0805
- removed X1: MICROSD, adafruit:MICROSD
- added C10, C11, C12: 0.1uf, SparkFun-Capacitors:0805
- added SJ10, SJ9: JUMPER-PAD-2-NC_BY_TRACE, SparkFun-Passives:PAD-JUMPER-2-NC_BY_TRACE_YES_SILK
- added U2, U3: (no value), SparkFun-DigitalIC:SO14
- added U4: USD-SOCKET, SparkFun-Connectors:MICROSD_1:1
- C9: value 10uF -> 0.1uf
- R23: value 2k -> 1k
- moved R30 390.6 mm to (56.2, 38.7), flipped to the bottom, turned to 180 degrees
- moved R29 386.3 mm to (56.2, 36.2), flipped to the bottom, turned to 180 degrees
- moved SJ6 379.8 mm to (54.9, 33.0), flipped to the bottom
- moved R26 375.5 mm to (87.6, 39.7), flipped to the bottom, turned to 270 degrees
- moved R28 375.1 mm to (87.6, 32.7), flipped to the bottom, turned to 270 degrees
- moved R27 375.1 mm to (87.6, 35.9), flipped to the bottom, turned to 270 degrees
- moved R17 366.4 mm to (81.9, 41.6), flipped to the bottom, turned to 270 degrees
- moved R18 365.7 mm to (81.9, 37.8), flipped to the bottom, turned to 270 degrees
- moved R25 365.6 mm to (81.9, 34.6), flipped to the bottom, turned to 270 degrees
- moved Q9 364.3 mm to (84.8, 39.7), flipped to the bottom, turned to 270 degrees
- moved C9 361.5 mm to (33.3, 38.4), turned to 90 degrees
- moved Q7 356.7 mm to (84.8, 35.9), flipped to the bottom, turned to 270 degrees
- moved Q8 356.4 mm to (84.8, 32.7), flipped to the bottom, turned to 270 degrees
- moved R6 248.8 mm to (87.6, 29.5), flipped to the bottom, turned to 270 degrees
- moved Q4 244.2 mm to (84.8, 29.5), flipped to the bottom, turned to 270 degrees
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Connections:
- removed net 12V: R23.1
- removed net ARM_SWITCH: JP9.VCC, R31.1, U1.30
- removed net CD: X1.CD1
- removed net N$12: D3.C, Q2.3
- removed net N$13: IC1.10, X1.5
- removed net N$14: IC1.12, R8.2, X1.2
- removed net N$16: IC1.6, X1.3
- removed net N$18: D5.C, Q5.3
- removed net N$19: D6.A, R11.2
- removed net N$20: D6.C, Q6.3
- removed net STATUS_LED_1: Q5.1, R7.1, U1.44
- removed net STATUS_LED_2: Q6.1, R10.1, U1.46
- removed net XBEE_RX: IC1.2, U$1.3
- removed net XBEE_TX: R2.1, U$1.2, U1.0
- new net SD_CS: U2.4, U4.2
- new net SD_DI: U2.5, U4.3
- new net SD_DO: U2.2, U4.7
- new net SD_SCK: U2.3, U4.5
- new net XBEE_RX_3V3: U$1.3, U3.2
- new net XBEE_TX_3V3: U$1.2, U3.3
- new net XBEE_TX_5V: Q1.1, R2.1, U1.0, U3.12
- net +3V3: now also C11.1, D2.A, D3.A, IMU_HEADER.1, SJ10.2, SJ9.2, U2.1, U3.1, U4.4; no longer IC1.1, IMU_HEADER.6, JP7.VCC, JP9.GND, R11.1, R3.1, R5.1, R9.1, X1.4
- net 5V: now also C10.1, C12.1, U2.14, U3.14
- net BATTVOLTAGE: now also U1.A0; no longer U1.A4
- net BUZZER: now also U1.36; no longer U1.42
- net CLK: now also U2.12; no longer IC1.14, IC1.9
- net CS: now also U2.11; no longer IC1.11
- net DI: now also U2.10; no longer IC1.7
- net DO: now also U2.13; no longer X1.7
- net GND: now also C10.2, C11.2, C12.2, IMU_HEADER.6, JP1.2, U2.7, U3.7, U4.6, U4.CD1, U4.CD2, U4.GND1, U4.GND3; no longer IC1.8, IMU_HEADER.1, JP1.1, Q5.2, Q6.2, R10.2, R31.2, R7.2, X1.6, X1.MT1, X1.MT2
- net G_RDY: now also IMU_HEADER.5, U1.28; no longer IMU_HEADER.4, U1.34
- net HOTWIRE_CONTINUITY: now also U1.A1; no longer U1.A6
- net L_RDY: now also IMU_HEADER.4, U1.26; no longer IMU_HEADER.5, U1.32
- net N$10: now also R3.1; no longer Q1.3
- net N$11: now also Q1.3, R3.2; no longer D3.A, R5.2
- net N$15: now also SJ9.1, U2.8; no longer D4.C, R8.1
- net N$17: now also SJ10.1, U3.8; no longer D5.A, R9.2
- net N$2: now also U3.4; no longer IC1.5
- net N$27: now also JP1.1; no longer JP1.2
- net N$4: now also D3.C, R5.1; no longer D4.A, IC1.15
- net N$8: no longer JP7.GND
- net N$9: now also Q2.3, R5.2; no longer D2.A, R3.2
- net PYRO_MONITOR: now also U1.A2; no longer U1.A5
- net RST_CTL: now also U1.9, U3.11; no longer IC1.4
- net STATUS_LED_BLUE: now also U1.34; no longer U1.40
- net STATUS_LED_GREEN: now also U1.30; no longer U1.36
- net STATUS_LED_RED: now also U1.32; no longer U1.38
- net V_BATT: now also R23.1
- net XBEE_RX_5V: now also Q2.1, U3.13; no longer IC1.3
Routing:
- net +3V3: track 6.37 -> 232.5 mm, vias 1 -> 7
- net 5V: track 23.0 -> 128.9 mm, vias 0 -> 4
- net SD_DO: track 0.00 -> 86.5 mm
- net SD_SCK: track 0.00 -> 85.2 mm
- net SD_DI: track 0.00 -> 84.8 mm, vias 0 -> 2
- net SD_CS: track 0.00 -> 82.6 mm
- net RST_CTL: track 0.00 -> 53.3 mm, vias 0 -> 3
- net SCL: track 0.00 -> 50.3 mm, vias 0 -> 2
- net XBEE_TX_5V: track 0.00 -> 48.3 mm
- net XBEE_RX_5V: track 0.00 -> 48.2 mm
- net HOTWIRE_CONTINUITY: track 0.00 -> 46.3 mm, vias 0 -> 2
- net XBEE_TX_3V3: track 0.00 -> 44.8 mm, vias 0 -> 2
- net SDA: track 0.00 -> 43.2 mm, vias 0 -> 1
- net L_RDY: track 0.00 -> 42.5 mm, vias 0 -> 1
- net XBEE_RX_3V3: track 0.00 -> 41.8 mm, vias 0 -> 4
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
Commit message: moved small things around added silk screen
Parts:
- added JP7: (no value), SparkFun-Connectors:1X02
- moved JP2 3.02 mm to (21.1, 4.60)
- moved D1 1.31 mm to (9.21, 17.5)
Routing:
- net HOTWIRE_CONTINUITY: track 46.3 -> 51.6 mm
- net V_BATT: track 82.8 -> 85.5 mm
- net N$1: track 2.55 -> 4.03 mm
- net N$5: track 18.3 -> 16.9 mm
- net N$6: track 6.70 -> 5.44 mm
- net GND: vias 47 -> 73
Other:
- board text added: "1"
- board text added: "2"
- board text added: "2S LIPO"
- board text added: "3"
- board text added: "3v3"
- board text added: "5v"
- board text added: "ALT_PYRO"
- board text added: "DO NOT CONFUSE"
- board text added: "GPS"
- board text added: "HOTWIRE"
- board text added: "IMU"
- board text added: "MICRO SD"
- board text added: "RSSI"
- board text added: "RX"
- board text added: "SERVOS"
- board text added: "TX"
- board text added: "V+"
- board text added: "V-"
- board text added: "VBat"
- board text added: "V_GOOD"
- board text added: "XBEE"

Commit message: Exported gerbers finished everything off. REV A
Parts:
- added U$7: (no value), RitLaunchInitiative:RITLAUNCH_LOGO_SMALLB
Routing:
- net GND: vias 73 -> 69
Other:
- board text added: "6/5/15"
- board text added: "Avionics Board"
- board text added: "Designed by:"
- board text added: "MIT Rocket Team"
- board text added: "REV: A"
- board text added: "Roy Cohen"
Changed lines of the file:
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@@
 <setting verticaltext="up"/>
 </settings>
-<grid distance="0.05" unitdist="inch" unit="inch" style="lines" multiple="1" display="no" altdistance="0.025" altunitdist="inch" altunit="inch"/>
+<grid distance="0.05" unitdist="inch" unit="inch" style="lines" multiple="1" display="no" altdistance="0.0125" altunitdist="inch" altunit="inch"/>
 <layers>
 <layer number="1" name="Top" color="4" fill="1" visible="yes" active="yes"/>
@@
 <wire x1="18.57375" y1="0.9525" x2="18.7325" y2="0.79375" width="0.3048" layer="21"/>
 <wire x1="8.73125" y1="1.5875" x2="8.255" y2="1.11125" width="0.3048" layer="21"/>
+<text x="73.66" y="22.86" size="1.27" layer="21" rot="R90">MIT Rocket Team</text>
+<text x="29.845" y="33.3375" size="1.016" layer="21">Avionics Board</text>
+<text x="29.845" y="30.7975" size="1.016" layer="21">Designed by:</text>
+<text x="29.845" y="28.575" size="1.016" layer="21">6/5/15</text>
+<text x="46.355" y="28.8925" size="1.016" layer="21">REV: A</text>
+<wire x1="29.845" y1="32.7025" x2="45.72" y2="32.7025" width="0.3048" layer="21"/>
+<wire x1="45.72" y1="32.7025" x2="46.0375" y2="33.02" width="0.3048" layer="21"/>
+<wire x1="29.845" y1="35.2425" x2="45.72" y2="35.2425" width="0.3048" layer="21"/>
+<wire x1="45.72" y1="35.2425" x2="48.26" y2="32.7025" width="0.3048" layer="21"/>
+<wire x1="48.26" y1="32.7025" x2="52.07" y2="32.7025" width="0.3048" layer="21"/>
+<wire x1="52.07" y1="32.7025" x2="52.705" y2="32.0675" width="0.3048" layer="21"/>
+<wire x1="52.705" y1="32.0675" x2="52.705" y2="28.2575" width="0.3048" layer="21"/>
+<wire x1="52.705" y1="28.2575" x2="52.3875" y2="27.94" width="0.3048" layer="21"/>
+<wire x1="52.3875" y1="27.94" x2="46.355" y2="27.94" width="0.3048" layer="21"/>
+<wire x1="46.355" y1="27.94" x2="45.085" y2="29.21" width="0.3048" layer="21"/>
+<wire x1="45.085" y1="29.21" x2="36.195" y2="29.21" width="0.3048" layer="21"/>
+<wire x1="36.195" y1="29.21" x2="34.925" y2="27.94" width="0.3048" layer="21"/>
+<wire x1="34.925" y1="27.94" x2="29.845" y2="27.94" width="0.3048" layer="21"/>
+<wire x1="29.845" y1="27.94" x2="29.5275" y2="28.2575" width="0.3048" layer="21"/>
+<wire x1="29.5275" y1="28.2575" x2="29.5275" y2="34.925" width="0.3048" layer="21"/>
+<wire x1="29.5275" y1="34.925" x2="29.845" y2="35.2425" width="0.3048" layer="21"/>
+<wire x1="71.4375" y1="41.275" x2="71.4375" y2="22.5425" width="0.3048" layer="21"/>
+<wire x1="71.4375" y1="22.5425" x2="72.0725" y2="21.9075" width="0.3048" layer="21"/>
+<wire x1="73.3425" y1="21.9075" x2="73.9775" y2="22.5425" width="0.3048" layer="21"/>
+<wire x1="73.9775" y1="22.5425" x2="73.9775" y2="41.275" width="0.3048" layer="21"/>
+<wire x1="73.9775" y1="41.275" x2="73.3425" y2="41.91" width="0.3048" layer="21"/>
+<wire x1="71.4375" y1="41.275" x2="72.0725" y2="41.91" width="0.3048" layer="21"/>
+<wire x1="34.6075" y1="10.795" x2="34.6075" y2="16.8275" width="0.3048" layer="21"/>
+<text x="39.37" y="30.48" size="1.4224" layer="21"> Roy Cohen</text>
 </plain>
 <attributes>
@@
 <attribute name="VALUE" x="31.75" y="5.715" size="1.27" layer="27" rot="R180"/>
 </element>
+<element name="U$7" library="RitLaunchInitiative" package="RITLAUNCH_LOGO_SMALLB" value="" x="81.28" y="16.51"/>
 </elements>
 <signals>
@@
 <via x="52.705" y="25.4" extent="1-16" drill="0.508"/>
 <via x="51.435" y="25.4" extent="1-16" drill="0.508"/>
-<wire x1="46.355" y1="25.4" x2="46.355" y2="25.4" width="0" layer="19" extent="1-16"/>
-<via x="47.625" y="27.94" extent="1-16" drill="0.508"/>
-<via x="48.895" y="27.94" extent="1-16" drill="0.508"/>
-<via x="50.165" y="27.94" extent="1-16" drill="0.508"/>
-<via x="46.355" y="29.21" extent="1-16" drill="0.508"/>
 <via x="33.02" y="22.5425" extent="1-16" drill="0.508"/>
 <via x="33.02" y="23.8125" extent="1-16" drill="0.508"/>
