File: Electronics/TelemetryBoard/RFModule900/RFModule900.sch (EAGLE design)
At the start: 34 parts

Commit message: more work on the RF 900mhz module
Parts:
- added C21: 1pF, SparkFun-Capacitors:CAP0402-CAP
- added C22, C23: 3pF, SparkFun-Capacitors:CAP0402-CAP
- added C24, C25: 4.3pF, SparkFun-Capacitors:CAP0402-CAP
- added C26, C27, C28: 56pF, SparkFun-Capacitors:CAP0402-CAP
- added C29: 3.9pF, SparkFun-Capacitors:CAP0402-CAP
- added C30: 5.6pF, SparkFun-Capacitors:CAP0402-CAP
- added C31: 22pF, SparkFun-Capacitors:CAP0402-CAP
- added C32: 1uF, SparkFun-Capacitors:10UF-16V-10%(TANT)
- added C34: 33pF, SparkFun-Capacitors:CAP0402-CAP
- added C35: 100pF, SparkFun-Capacitors:CAP0402-CAP
- added C36: 100nF, SparkFun-Capacitors:CAP0402-CAP
- added C37: 2.2uF, SparkFun-Capacitors:CAP0402-CAP
- added L10: 12nH, SparkFun-Passives:INDUCTOR0402
- added L11: 10nH, SparkFun-Passives:INDUCTOR0402
- added L6: 18nH, SparkFun-Passives:INDUCTOR0402
- added L7: 22nH, SparkFun-Passives:INDUCTOR0402
- added L8: 8.2nH, SparkFun-Passives:INDUCTOR0402
- added L9: 100nH, SparkFun-Passives:INDUCTOR0402
- added R5, R6, R7: 5k, SparkFun-Resistors:RESISTOR0402
- added SJ2: JUMPER-PAD-3-2OF3_NC_BY_TRACE_SMALL, SparkFun-Passives:JUMPER-PAD-3-2OF3_NC_BY_TRACE_SMALL
- added Y1: 30 Mhz, RitLaunchInitiative:CRYSTAL
- C1: value 7.5pF -> 2.7pF
- C11: value 1uF -> 10uF
- C16: value 10uF -> 1uF
- C19: value 1uF -> 22pF
- C2: value 39pF -> 1uF
- C8: value 39pF -> 22pF
- L1: value 2.7nH -> 10nH
- L4, L5: value BLM15HB121SN1 -> (none)
Connections:
- removed net N$2 (its old number): C1.2, U$2.RF_IN
- new net 3V1: C32.+, U$4.V_OUT
- new net 5V: R5.1, U$4.VIN
- new net N$12: C21.1, L6.1, U$1.RX_P
- new net N$13: C21.2, C23.2, L7.2
- new net N$14: C23.1, C28.2
- new net N$15: C25.2, L8.2, X1.ANT
- new net N$16: C26.2, U$3.RFC
- new net N$19: C11.1, C2.1, R1.1
- new net N$20: C29.1, L9.2, U$1.TX
- new net N$21: C29.2, L10.1
- new net N$22: C30.2, L1.1, L10.2
- new net N$23: C27.1, U$3.RF1
- new net N$24: C28.1, U$3.RF2
- new net N$25: R6.1, SJ2.2
- new net N$26: C19.2, R6.2, U$3.LS
- new net N$27: C22.2, L6.2, L7.1, U$1.RX_N
- new net N$28: U$1.XIN, Y1.P$1
- new net N$29: U$1.XOUT, Y1.P$2
- new net N$4: C16.1, R4.2, U$2.PWR_SENSE
- new net RADIO_ENABLE: R7.2, U$1.SDN
- new net TR_SWITCH_CTL: C31.2, U$1.GPIO3, U$3.CTL
- net 3.3V: now also C34.2, C35.2, C36.2, C37.2, C8.2, L9.1, SJ2.3, U$1.VDD, U$3.VDD
- net GND: now also C1.1, C16.2, C19.1, C2.2, C22.1, C24.1, C25.1, C30.1, C31.1, C32.-, C34.1, C35.1, C36.1, C37.1, C8.1, R7.1, SJ2.1, U$1.GND, U$3.GND, U$4.GND; no longer C16.1, C19.2, L1.2
- net N$1: now also C1.2, L1.2, L11.1; no longer C1.1, C2.2, L1.1
- net N$10: now also C24.2, C26.1, L8.1; no longer U$3.RFC, X1.ANT
- net N$17: now also L11.2, U$2.RF_IN; no longer C19.1, R4.2, U$2.PWR_SENSE
- net N$3: now also C12.1, C17.1, R2.1; no longer C2.1
- net N$5: now also C27.2; no longer C8.2
- net N$7: now also R5.2, U$4.V_EN; no longer C11.1, C12.1, C16.2, C17.1, R1.1, R2.1
Other:
- note added: "Choke"
- note added: "LowPass Filter"
- note added: "Lowpass"
- note added: "T/R switch"
- note added: "TX match"
- note added: "reciever input match"
- moved on the sheet: C1, C10, C11, C12, C13, C14, C15, C16, C17, C18, C19, C2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

Commit message: adding status leds and power sequencing as well as clean up
Parts:
- added D1, D2, D3, D4, D5: (no value), SparkFun-LED:LED0603
- added JP1: (no value), SparkFun-Connectors:M10X2SPECIAL
- added JP2, JP3: (no value), SparkFun-Connectors:M05X2PTH
- added R10, R11, R12, R14, R15, R8, R9: 5k, SparkFun-Resistors:RESISTOR0402
- added R13: 10k, SparkFun-Resistors:RESISTOR0402
- added U$5: AO6602, RitLaunchInitiative:AO6602
- added U1, U2: TPS2561, RitLaunchInitiative:TPS2561
- SJ2: value JUMPER-PAD-3-2OF3_NC_BY_TRACE_SMALL -> invert Control Signal
Connections:
- new net 3V3_MAIN: R13.2
- new net GPIO0: U$1.GPIO0
- new net GPIO1: U$1.GPIO1
- new net GPIO2: U$1.GPIO2
- new net N$11: R9.2, U1.ILIM
- new net N$30: D2.C, R10.2
- new net N$31: D1.C, R12.2
- new net N$32: R8.2, U2.ILIM
- new net N$33: D5.A, R5.2
- new net N$34: D5.C, U$5.D1
- new net N$35: D4.A, U$5.S2
- new net N$36: D4.C, R15.1
- new net N_IRQ: JP1.11, U$1.N_IRQ
- new net N_SEL: JP1.19, U$1.N_SEL
- new net PA_3V3: C14.2, C15.1, C20.1, D2.A, L4.2, L5.2, R3.1, R4.1, U$2.VCC1, U$2.VCC_BIAS, U2.OUT1, U2.OUT2
- new net PA_ENABLE: JP1.20, U$4.V_EN, U2.EN1, U2.EN2
- new net PA_TEMP: JP1.14, R13.1, R14.2
- new net RADIO_3V3: C34.2, C35.2, C36.2, C37.2, D1.A, L9.1, U$1.VDD, U1.OUT1
- new net SCLK: JP1.13, U$1.SCLK
- new net SDI: JP1.17, U$1.SDI
- new net SDO: JP1.15, U$1.SDO
- new net STATUS_LED: JP1.16
- net 3.3V: now also JP1.1, JP1.2, JP1.3, JP1.4, JP1.6, R5.1, U$5.D2, U1.IN, U2.IN; no longer C14.2, C15.1, C20.1, C34.2, C35.2, C36.2, C37.2, L4.2, L5.2, L9.1, R3.1, R4.1, U$1.VDD, U$2.VCC1, U$2.VCC_BIAS
- net 3V1: now also D3.A
- net 5V: now also JP1.9; no longer R5.1
- net GND: now also JP1.10, JP1.12, JP1.5, JP1.7, JP1.8, R10.1, R11.1, R12.1, R14.1, R15.2, R8.1, R9.1, U$5.S1, U1.GND, U2.GND, Y1.GND
- net N$7: now also D3.C, R11.2; no longer R5.2, U$4.V_EN
- net RADIO_ENABLE: now also JP1.18, U1.EN1
- net TR_SWITCH_CTL: now also U$5.G1, U$5.G2
Other:
- note added: "3.3v tollerant"
- note added: "<- RF ->"
- note added: "<- RF IN"
- note added: "Antenna"
- note added: "MAIN RF TRANSCEIVER"
- note added: "MAIN TRANSCEIVER POWER MANAGMENT"
- note added: "RF OUT ->"
- note added: "RF PA Power MANAGMENT"
- note added: "RF POWER AMPLIFIER"
- note added: "TRANSMIT RECEIVE SWITCH"
- note added: "Thermistor"
- note added: "sma connector"
- moved on the sheet: C1, C10, C11, C12, C13, C14, C15, C16, C17, C18, C19, C2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

Commit message: Cleaning more things up
Parts:
- added R16, R17: 10k, SparkFun-Resistors:RESISTOR0402
Connections:
- net GND: now also R16.2
Other:
- note added: "Add more tantilum caps for decoupling on both major IC's"
- note added: "Breakout GPIO's"
- note added: "Calculate resistors for led current limiiting"
- note added: "Finalize Connector configuration for daughter board interface"
- note added: "Find Model Number of thermistor"
- note added: "Set resistor values for Current Limits on Load switches"
- note added: "TODO"
- note added: "TX RX status led"
- note added: "Try finding The proper values for the two Ferrites L4 L5"
- moved on the sheet: C32, D2, D3, D4, D5, R10, R11, R15, R5, R8, U$4, U$5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
