File: Electronics/TelemetryBoard/RFModule900/RFModule900_Mark1.sch (EAGLE design)
At the start: 82 parts, among them U1 TPS2561, U2 TPS2561, Y1 30 Mhz

Commit message: More work on RF card
Parts:
- added C33: 0.01uF, SparkFun-Capacitors:CAP0402-CAP
- C11, C15, C17: device SparkFun-Capacitors:CAP0402-CAP -> SparkFun-Capacitors:10UF-16V-10%(TANT); DIGI (none) -> 399-3678-1-ND; MPN (none) -> T491A105K016AT
- L4, L5: value (none) -> 260; device inductors:BLM15HB121SN1 -> SparkFun-Passives:INDUCTOR0603; MPN (none) -> BLM18EG221SN1D
Connections:
- net GND: now also C11.-, C15.-, C17.-, C33.1; no longer C11.2, C15.2, C17.2
- net N$19: now also C11.+; no longer C11.1
- net N$3: now also C17.+; no longer C17.1
- net N$6: now also L4.2, L5.2; no longer L4.1, L5.1
- net PA_3V3: now also C15.+, C33.2, L4.1, L5.1; no longer C15.1, L4.2, L5.2

Commit message: adding directional couplers to board
Parts:
- added C38, C41: 0.1uF, SparkFun-Capacitors:CAP0402-CAP
- added C39, C40, C42, C43: DNP, SparkFun-Capacitors:CAP0402-CAP
- added L12, L13: 0 ohm, SparkFun-Passives:INDUCTOR0402
- added R18, R19: 5k, SparkFun-Resistors:RESISTOR0402
- added T1, T2: DC08-73, RitLaunchInitiative:DC08-73
- added U$6: TL331-Q1, RitLaunchInitiative:TL331-Q1
- added U$7: SN74AHC1G08, RitLaunchInitiative:SN74AHC1G08
- added U$8: SN74LVC1G14, RitLaunchInitiative:SN74LVC1G14
- added U$9: SN74LVC1G32, RitLaunchInitiative:SN74LVC1G32
- added U3: LMV321, RitLaunchInitiative:LMV321
- added U4, U5: LTC5505, RitLaunchInitiative:LTC5505
- added U6: MCP4728, RitLaunchInitiative:MCP4728
Connections:
- new net N$37: R18.1, U4.SHDN
- new net N$38: U$8.O, U$9.I0
- new net N$39: C40.2, L12.1, T1.COUPLED
- new net N$40: C39.2, L12.2, U4.RF_IN
- new net N$41: T1.OUT, T2.OUT
- new net N$42: R19.1
- new net N$43: C43.2, L13.1, U5.RF_IN
- new net N$44: C42.2, L13.2, T2.COUPLED
- new net N$45: T2.IN, X1.ANT
- new net N$46: U$7.I0, U$9.O
- new net N$47: U$7.I1
- new net RF_POWER_IN: U5.VOUT
- new net RF_POWER_OUT: U4.VOUT
- net 3.3V: now also C38.1, C41.1, R18.2, R19.2, U$6.GND, U$8.GND, U$9.GND, U4.VCC
- net GND: now also C38.2, C39.1, C40.1, C41.2, C42.1, C43.1, T1.GND, T2.GND, U$6.VCC, U$7.VCC, U$8.VCC, U$9.VCC, U4.GND
- net N$15: no longer X1.ANT
Other:
- note added: "A(C + !B)"
- note added: "A: PA_Enable"
- note added: "B: VSWR _FAULT"
- note added: "C: PA_OVERRIDE"
- note added: "Subtractor"
- moved on the sheet: X1

Commit message: Routing RF path
Parts:
- removed U3: LMV321, RitLaunchInitiative:LMV321
- removed X1: (no value), adafruit:SMACONNECTOR
- added C44, C45, C46, C47, C48: 0.1uF, SparkFun-Capacitors:CAP0402-CAP
- added R20, R21: 5k, SparkFun-Resistors:RESISTOR0402-RES
- added U$10: 0732511150_SMA_EDGE_LAUNCH, RitLaunchInitiative:0732511150_SMA_EDGE_LAUNCH
- added U7: LMV321, RitLaunchInitiative:LMV321
- JP1: value (none) -> M10X2SPECIAL
- JP2, JP3: value (none) -> M05X2PTH
- R1, R10, R11, R12, R13, R14, R15, R16, R17, R18, R19, R2, R3, R4, R5, R6, R7, R8, R9: device SparkFun-Resistors:RESISTOR0402 -> SparkFun-Resistors:RESISTOR0402-RES
Connections:
- new net N$48: R20.1, R21.2, U7.IN-
- new net N$51: U$6.OUT, U$8.I
- new net PA_LOADSWITCH_ENABLE: U$4.V_EN, U$7.O, U2.EN1, U2.EN2
- new net PA_OVERRIDE: U$9.I1
- new net REFLECTED_POWER_REF: U$6.IN-
- net 3.3V: now also C44.2, C45.2, C46.2, C47.2, C48.1, U$7.GND, U5.VCC, U7.GND
- net GND: now also C44.1, C45.1, C46.1, C47.1, C48.2, R21.1, U$10.GND, U5.GND, U7.VCC; no longer X1.GND1, X1.GND2, X1.GND3, X1.GND4
- net N$14: now also C27.2; no longer C28.2
- net N$15: now also T1.IN
- net N$42: now also U5.SHDN
- net N$45: now also U$10.1; no longer X1.ANT
- net N$47: now also R20.2, U$6.IN+, U7.OUT; no longer U$7.I1
- net N$5: now also C28.2; no longer C27.2
- net PA_ENABLE: now also U$7.I1; no longer U$4.V_EN, U2.EN1, U2.EN2
- net RF_POWER_IN: now also U7.IN+
Other:
- note removed: "Subtractor"
- moved on the sheet: C27, C28, U$8

Commit message: wiring in dac
Parts:
- added C49, C50: 10uF, SparkFun-Capacitors:10UF-16V-10%(TANT)
- added SJ1, SJ3, SJ4: JUMPER-PAD-3-2OF3_NC_BY_TRACE_LARGE, SparkFun-Passives:JUMPER-PAD-3-2OF3_NC_BY_TRACE_LARGE
- C11: value 10uF -> 0.1uF; device SparkFun-Capacitors:10UF-16V-10%(TANT) -> SparkFun-Capacitors:CAP0402-CAP; DIGI 399-3678-1-ND -> (none); MPN T491A105K016AT -> (none)
- C17: value 10uF -> 2.2uF; device SparkFun-Capacitors:10UF-16V-10%(TANT) -> SparkFun-Capacitors:CAP0402-CAP; DIGI 399-3678-1-ND -> (none); MPN T491A105K016AT -> (none)
Connections:
- net N$18 renamed PA_PWR_REF
- net N$4 renamed PA_PWR_SENSE
- removed net 3V3_MAIN: R13.2
- removed net N$3: C12.1, C17.+, R2.1
- new net N$4: C12.1, C50.+, R2.1, SJ3.2
- new net N$49: C11.1, C17.2, SJ4.2, U6.VDD
- new net SCL: U6.SCL
- new net SDA: U6.SDA
- new net VREG1_DAC: SJ1.3, U6.VOUT_B
- new net VREG2_DAC: SJ3.3, U6.VOUT_C
- net 3.3V: now also C44.1, C45.1, C46.1, C47.1, R13.2, SJ4.3, U$6.VCC, U$7.VCC, U$8.VCC, U$9.VCC, U7.VCC; no longer C44.2, C45.2, C46.2, C47.2, U$6.GND, U$7.GND, U$8.GND, U$9.GND, U7.GND
- net 3V1: now also SJ1.1, SJ3.1
- net 5V: now also SJ4.1
- net GND: now also C11.2, C17.1, C44.2, C45.2, C46.2, C47.2, C49.-, C50.-, U$6.GND, U$7.GND, U$8.GND, U$9.GND, U6.LDAC, U6.VSS, U7.GND; no longer C11.-, C17.-, C44.1, C45.1, C46.1, C47.1, U$6.VCC, U$7.VCC, U$8.VCC, U$9.VCC, U7.VCC
- net N$19: now also C49.+, SJ1.2; no longer C11.+
- net REFLECTED_POWER_REF: now also U6.VOUT_A
Other:
- note added: "Signal amplification"
- note added: "Threshold comparason"
- note added: "VSWR Hardware breaker"
- note added: "Will fix this later in footprint"
- moved on the sheet: C21, C22, C23, C34, C35, C36, C37, C44, C45, C46, C47, C48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

Commit message: organizing schema and adding dac power control
Also adding power fault feedback on all load switches
Parts:
- removed C12: 1uF, SparkFun-Capacitors:CAP0402-CAP
- removed D1, D2: (no value), SparkFun-LED:LED0603
- added C51, C52, C53, C54: 0.1uF, SparkFun-Capacitors:CAP0402-CAP
- added C55: 1uF, SparkFun-Capacitors:CAP0402-CAP
- added D6, D8, D9: (no value), SparkFun-LED:LED0603
- added JP4: (no value), SparkFun-Connectors:M01PTH
- added R22, R23: DNP, SparkFun-Resistors:RESISTOR0402-RES
- added R24: 5k, SparkFun-Resistors:RESISTOR0402-RES
- added R25, R26, R27: 100k, SparkFun-Resistors:RESISTOR0402-RES
- added SJ5: JUMPER-PAD-3-2OF3_NC_BY_TRACE_SMALL, SparkFun-Passives:JUMPER-PAD-3-2OF3_NC_BY_TRACE_SMALL
- added U$11: SN74LVC1G14, RitLaunchInitiative:SN74LVC1G14
- C14: device SparkFun-Capacitors:CAP0402-CAP -> SparkFun-Capacitors:CAP0805; DIGI (none) -> 712-1398-1-ND
- C16, C2: DIGI (none) -> 587-1453-1-ND; MPN (none) -> JMK105BJ225MVHF
- C20, C56: DIGI (none) -> 490-3890-1-ND; MPN (none) -> GRM155R61A105KE15D
- C3: DIGI (none) -> 712-1261-1-ND; MPN (none) -> 500R07S150JV4TD
- C4: DIGI (none) -> 712-1257-1-ND; MPN (none) -> 500R07S120JV4TD
- C5: DIGI (none) -> 712-1253-1-ND; MPN (none) -> 500R07S100JV4TD
- C6: MOUSER (none) -> 609-500R07S5R6BV4T; MPN (none) -> 500R07S5R6BV4
- C7: DIGI (none) -> 712-1162-1-ND; MPN (none) -> 500R07S0R5BV4TD
- C9: DIGI (none) -> 712-1277-1-ND
- D3: COLOR (none) -> Red; DIGI (none) -> 160-1447-1-ND
- D4: COLOR (none) -> Green; DIGI (none) -> 160-1446-1-ND
- D5: COLOR (none) -> Blue; DIGI (none) -> 160-1647-1-ND
- L2: device SparkFun-Passives:INDUCTOR0402 -> SparkFun-Passives:INDUCTOR0603; MPN (none) -> LL1608-FSL1N5S; RICHARDSON_RFPD (none) -> http://www.richardsonrfpd.com/pages/Product-Details.aspx?pr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
- L4, L5: DIGI (none) -> 490-3992-1-ND
- R10, R15, R5: value 5k -> 270
- R11: value 5k -> 220
- R16, R17: value 10k -> DNP
- R8, R9: value 5k -> 25.5k
- SJ1, SJ3, SJ4: value JUMPER-PAD-3-2OF3_NC_BY_TRACE_LARGE -> JUMPER-PAD-3-2OF3_NC_BY_TRACE_SMALL; device SparkFun-Passives:JUMPER-PAD-3-2OF3_NC_BY_TRACE_LARGE -> SparkFun-Passives:JUMPER-PAD-3-2OF3_NC_BY_TRACE_SMALL
- U$2: DIGI (none) -> 689-1091-1-ND
- U$4: value LP3984 -> LP3984_DNP
- renumbered C18 to C56
Connections:
- net PA_LOADSWITCH_ENABLE renamed PA_PWR_EN_BREAKER
- net PA_OVERRIDE renamed PA_BREAKER_OVERRIDE
- removed net PA_ENABLE: JP1.20, U$7.I1
- removed net RADIO_ENABLE: JP1.18, R7.2, U$1.SDN, U1.EN1
- removed net STATUS_LED: JP1.16
- new net BUFF_TR_SWITCH_CTL: R16.1, U$11.O, U$5.G1
- new net DAC_3V3: D8.A, SJ5.3, U1.OUT2
- new net DAC_PWR_EN: U1.EN2
- new net DAC_PWR_FAULT: R26.1, U1.FAULT2
- new net N$18: JP4.1, U6.VOUT_D
- new net N$50: D9.C, R12.2
- new net N$52: R17.1, U$5.G2
- new net N$53: SJ4.3, SJ5.2
- new net PA_PWR_EN: U$7.I1
- new net PA_PWR_FAULT: R27.1, U2.FAULT1, U2.FAULT2
- new net RADIO_PWR_EN: U1.EN1
- new net RADIO_PWR_FAULT: R25.1, U1.FAULT1
- new net RADIO_SHUTDOWN: R7.2, U$1.SDN
- net 3.3V: now also C51.1, C52.1, C53.1, R17.2, R22.2, R23.2, R25.2, R26.2, R27.2, SJ5.1, U$11.VCC; no longer SJ4.3
- net 5V: now also C54.2
- net GND: now also C51.2, C52.2, C53.2, C54.1, C55.2, R24.1, U$11.GND; no longer C12.2
- net N$19: now also C16.1; no longer C2.1
- net N$30: now also D6.C; no longer D2.C
- net N$31: now also D8.C, R24.2; no longer D1.C, R12.2
- net N$4: now also C2.1; no longer C12.1
- net N_IRQ: no longer JP1.11
- net N_SEL: no longer JP1.19
- net PA_3V3: now also D6.A; no longer D2.A
- net PA_PWR_SENSE: now also C55.1; no longer C16.1
- net PA_TEMP: no longer JP1.14
- net RADIO_3V3: now also D9.A; no longer D1.A
- net SCL: now also R22.1
- net SCLK: no longer JP1.13
- net SDA: now also R23.1
- net SDI: no longer JP1.17
- net SDO: no longer JP1.15
- net TR_SWITCH_CTL: no longer U$5.G1, U$5.G2
Other:
- note added: "2 AMP current limit per channel"
- note added: "A"
- note added: "Add Temp sensor LM75B"
- note added: "B"
- note added: "Buffering TR_SWITCH_CTL"
- note added: "C"
- note added: "Complementary Fet array"
- note added: "Optional input attenuation"
- note added: "POWER MANAGMENT"
- note added: "R16/R17 in case active low and high signal does not turn off the complementary fets"
- note added: "VSWR Measurement"
- note removed: "MAIN TRANSCEIVER POWER MANAGMENT"
- note removed: "RF PA Power MANAGMENT"
- moved on the sheet: C11, C16, C17, C2, C44, C45, C46, C47, C48, D4, D5, R10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

Commit message: changed to a 3.6v bus for main board power for amp
Parts:
- removed C48: 0.1uF, SparkFun-Capacitors:CAP0402-CAP
- removed U7: LMV321, RitLaunchInitiative:LMV321
- added C12: 0.1uF, SparkFun-Capacitors:CAP0402-CAP
- added R28: 10k, SparkFun-Resistors:RESISTOR0402
- added U$16: 10k, RitLaunchInitiative:THERMISTOR
- added U3: LM75B, RitLaunchInitiative:LM75B
- JP1: value M10X2SPECIAL -> (none)
- JP2, JP3: value M05X2PTH -> (none)
- R1, R10, R11, R15, R16, R17, R18, R19, R2, R22, R23, R25, R26, R27, R3, R4, R5, R6, R7, R8, R9: device SparkFun-Resistors:RESISTOR0402-RES -> SparkFun-Resistors:RESISTOR0402
- R12, R24: value 5k -> 270; device SparkFun-Resistors:RESISTOR0402-RES -> SparkFun-Resistors:RESISTOR0402
- R13: value 10k -> 0; device SparkFun-Resistors:RESISTOR0402-RES -> SparkFun-Resistors:RESISTOR0402
- R14, R21: value 5k -> DNP; device SparkFun-Resistors:RESISTOR0402-RES -> SparkFun-Resistors:RESISTOR0402
- R20: value 5k -> 0; device SparkFun-Resistors:RESISTOR0402-RES -> SparkFun-Resistors:RESISTOR0402
Connections:
- net N$51 renamed VSWR_BREAKER_STATE
- net PA_3V3 renamed PA_3V6
- new net 3.6V: C52.1, U2.IN
- net 3.3V: now also C12.2, R28.2, U3.VCC; no longer C48.1, C52.1, R13.2, U2.IN, U7.VCC
- net GND: now also C12.1, R14.2, R21.2, U$16.2, U3.GND; no longer C48.2, R14.1, R21.1, U7.GND
- net N$47: now also C55.1, R13.1, R4.2, U$2.PWR_SENSE; no longer R20.2, U$6.IN+, U7.OUT
- net N$48: now also C56.1, R3.2, U$2.PWR_REF; no longer R21.2, U7.IN-
- net PA_PWR_REF: now also R20.2, R21.1; no longer C56.1, R3.2, U$2.PWR_REF
- net PA_PWR_SENSE: now also R13.2, R14.1; no longer C55.1, R4.2, U$2.PWR_SENSE
- net PA_TEMP: now also R28.1, U$16.1; no longer R13.1, R14.2
- net RF_POWER_IN: now also U$6.IN+; no longer U7.IN+
- net SCL: now also U3.SCL
- net SDA: now also U3.SDA
Other:
- note added: "1.75v"
- note added: "Add ADC ADC128D818CIMTX/NOPB"
- note added: "Divide sense voltages down to bring into ADC input range"
- note added: "I2C adress:"
- note added: "add MIC5504-3.3YM5 TR LDO as 3v3 supply"
- note removed: "Signal amplification"
- note removed: "Thermistor"
- moved on the sheet: R13, R14, R17, R20, R21

Commit message: added new switching regulator
Parts:
- added U$15: LMZ31704, RitLaunchInitiative:LMZ31704
- added U7: ADC128D818, RitLaunchInitiative:ADC128D818
- added U8: MIC5504-3.3YM5, RitLaunchInitiative:MIC5504-3.3YM5
Other:
- note added: "576-4310-1-ND"
- note added: "576-4764-1-ND"
- note added: "Add switching supply to bring 12v to 3.6 lmz31704"
Changed lines of the file:
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@@
 </part>
 <part name="R28" library="SparkFun-Resistors" deviceset="RESISTOR" device="0402" value="10k"/>
+<part name="U7" library="RitLaunchInitiative" deviceset="ADC128D818" device=""/>
+<part name="U$15" library="RitLaunchInitiative" deviceset="LMZ31704" device=""/>
+<part name="U8" library="RitLaunchInitiative" deviceset="MIC5504-3.3YM5" device=""/>
 </parts>
 <sheets>
@@
 <wire x1="307.34" y1="93.98" x2="307.34" y2="210.82" width="0.1524" layer="94"/>
 <wire x1="307.34" y1="210.82" x2="12.7" y2="210.82" width="0.1524" layer="94"/>
-<wire x1="-22.86" y1="368.3" x2="266.7" y2="368.3" width="0.1524" layer="94"/>
+<wire x1="-210.82" y1="368.3" x2="266.7" y2="368.3" width="0.1524" layer="94"/>
 <wire x1="266.7" y1="368.3" x2="266.7" y2="226.06" width="0.1524" layer="94"/>
-<wire x1="266.7" y1="226.06" x2="-22.86" y2="226.06" width="0.1524" layer="94"/>
-<wire x1="-22.86" y1="226.06" x2="-22.86" y2="368.3" width="0.1524" layer="94"/>
+<wire x1="266.7" y1="226.06" x2="-210.82" y2="226.06" width="0.1524" layer="94"/>
+<wire x1="-210.82" y1="226.06" x2="-210.82" y2="368.3" width="0.1524" layer="94"/>
 <text x="127" y="213.36" size="3.81" layer="94">RF POWER AMPLIFIER</text>
 <wire x1="-231.14" y1="162.56" x2="-53.34" y2="162.56" width="0.1524" layer="94"/>
@@
 <text x="756.92" y="78.74" size="3.81" layer="94">sma connector</text>
 <text x="535.94" y="45.72" size="1.6764" layer="94">TX RX status led</text>
-<text x="-208.28" y="350.52" size="5.08" layer="94">TODO</text>
-<text x="-208.28" y="381" size="2.1844" layer="94">Set resistor values for Current Limits on Load switches</text>
-<text x="-208.28" y="378.46" size="2.1844" layer="94">Calculate resistors for led current limiiting</text>
-<text x="-208.28" y="342.9" size="2.1844" layer="94">Add more tantilum caps for decoupling on both major IC's </text>
-<text x="-208.28" y="337.82" size="2.1844" layer="94">Find Model Number of thermistor</text>
-<text x="-208.28" y="335.28" size="2.1844" layer="94">Finalize Connector configuration for daughter board interface</text>
-<text x="-208.28" y="332.74" size="2.1844" layer="94">Breakout GPIO's </text>
-<text x="-208.28" y="373.38" size="2.1844" layer="94">Try finding The proper values for the two Ferrites L4 L5</text>
+<text x="-330.2" y="388.62" size="5.08" layer="94">TODO</text>
+<text x="-330.2" y="419.1" size="2.1844" layer="94">Set resistor values for Current Limits on Load switches</text>
+<text x="-330.2" y="416.56" size="2.1844" layer="94">Calculate resistors for led current limiiting</text>
+<text x="-330.2" y="381" size="2.1844" layer="94">Add more tantilum caps for decoupling on both major IC's </text>
+<text x="-330.2" y="378.46" size="2.1844" layer="94">Find Model Number of thermistor</text>
+<text x="-330.2" y="375.92" size="2.1844" layer="94">Finalize Connector configuration for daughter board interface</text>
+<text x="-330.2" y="373.38" size="2.1844" layer="94">Breakout GPIO's </text>
+<text x="-330.2" y="411.48" size="2.1844" layer="94">Try finding The proper values for the two Ferrites L4 L5</text>
 <text x="-43.18" y="76.2" size="3.81" layer="94">&lt;- RF IN </text>
 <text x="-48.26" y="119.38" size="3.81" layer="94">RF OUT -&gt; </text>
@@
 <text x="401.32" y="363.22" size="3.81" layer="91">VSWR Hardware breaker</text>
 <text x="411.48" y="353.06" size="1.778" layer="91">Threshold comparason</text>
-<text x="-208.28" y="375.92" size="1.778" layer="91">Add Temp sensor LM75B</text>
+<text x="-330.2" y="414.02" size="1.778" layer="91">Add Temp sensor LM75B</text>
 <text x="477.52" y="297.18" size="2.54" layer="91">C</text>
 <text x="441.96" y="317.5" size="2.54" layer="91">B</text>
@@
 <text x="-35.56" y="-116.84" size="1.016" layer="91">1.75v</text>
 <text x="66.04" y="167.64" size="1.4224" layer="91">Divide sense voltages down to bring into ADC input range</text>
-<text x="-208.28" y="327.66" size="1.4224" layer="91">Add ADC ADC128D818CIMTX/NOPB</text>
-<text x="-208.28" y="330.2" size="1.4224" layer="91">add MIC5504-3.3YM5 TR LDO as 3v3 supply</text>
+<text x="-330.2" y="406.4" size="1.4224" layer="91">Add ADC ADC128D818CIMTX/NOPB</text>
+<text x="-330.2" y="408.94" size="1.4224" layer="91">add MIC5504-3.3YM5 TR LDO as 3v3 supply</text>
 <text x="50.8" y="203.2" size="1.4224" layer="91">I2C adress:</text>
 <text x="177.8" y="353.06" size="1.4224" layer="91">I2C adress:</text>
+<text x="-276.86" y="396.24" size="1.4224" layer="91">576-4310-1-ND</text>
+<text x="-276.86" y="393.7" size="1.4224" layer="91">576-4764-1-ND</text>
+<text x="-330.2" y="358.14" size="1.778" layer="91">Add switching supply to bring 12v to 3.6 lmz31704</text>
 </plain>
 <instances>
@@
 </instance>
 <instance part="R28" gate="G$1" x="40.64" y="167.64" rot="R90"/>
+<instance part="U7" gate="G$1" x="-127" y="347.98"/>
+<instance part="U$15" gate="G$1" x="-129.54" y="302.26"/>
+<instance part="U8" gate="G$1" x="-129.54" y="256.54"/>
 </instances>
 <busses>
@@
 </segment>
 </net>
+<net name="N$51" class="0">
+<segment>
+<wire x1="-281.686" y1="397.002" x2="-277.114" y2="397.002" width="0.1524" layer="91"/>
+<wire x1="-277.114" y1="397.002" x2="-277.114" y2="392.43" width="0.1524" layer="91"/>
+<wire x1="-277.114" y1="392.43" x2="-262.636" y2="392.43" width="0.1524" layer="91"/>
+<wire x1="-262.636" y1="392.43" x2="-262.636" y2="398.272" width="0.1524" layer="91"/>
+<wire x1="-262.636" y1="398.272" x2="-277.114" y2="398.272" width="0.1524" layer="91"/>
+<wire x1="-277.114" y1="398.272" x2="-277.114" y2="397.002" width="0.1524" layer="91"/>
+</segment>
+</net>
