File: Electronics/TelemetryBoard/RFModule900/RFModule900_Mark1.sch (EAGLE design)
At the start: 134 parts, among them T1 DC08-73, T2 DC08-73, U1 TPS2561, U2 TPS2561, U3 LM75B, U4 LTC5505, U5 LTC5505, U6 MCP4728, U7 ADC128D818, U8 MIC5504-3.3YM5, Y1 30 Mhz

Commit message: wiring up new buck and 3.3v ldo
Parts:
- removed JP2, JP3: (no value), SparkFun-Connectors:M05X2PTH
- added C18, C57, C61: 100uF, SparkFun-Retired:2.2UF-CERCAP-10009
- added C48, C58: 100uF, RitLaunchInitiative:C1210C107M4PAC7800
- added C59: 47uF, RitLaunchInitiative:GRM32ER61C476KE15K
- added C60, C64, C66: 0.1uF, SparkFun-Capacitors:CAP0402-CAP
- added C62, C63, C65: 1uF, SparkFun-Capacitors:CAP0402-CAP
- added D1, D2: (no value), SparkFun-LED:LED0603
- added R29: 287, SparkFun-Resistors:RESISTOR0402
- added R30: 90.9k, SparkFun-Resistors:RESISTOR0402
- added R31, R32, R33: 270, SparkFun-Resistors:RESISTOR0402
- added R34, R35: 5k, SparkFun-Resistors:RESISTOR0402
- C32: value 1uF -> DNP
- C54: value 0.1uF -> DNP
- D3: value (none) -> DNP
- R11: value 220 -> DNP
Connections:
- new net 12V: C48.1, C58.1, C59.1, C60.1, U$15.PVIN, U$15.VIN
- new net 3V6_PWRGD: U$15.PWRGD
- new net ADC_INT: U7.INT
- new net N$54: R29.2, U$15.VADJ
- new net N$55: R30.2, U$15.RT_CLK
- new net N$56: D2.C, R32.2
- new net N$57: R33.2, U8.EN
- new net N$58: D1.C, R31.2
- new net N$59: R35.2, U7.A1
- new net N$60: R34.2, U7.A0
- net 3.3V: now also C63.1, C65.1, C66.1, D2.A, U7.VCC, U8.VOUT
- net 3.6V: now also C18.1, C57.1, C61.1, C62.2, C64.1, D1.A, R33.1, U$15.SENSE+, U$15.VOUT, U8.VIN
- net GND: now also C18.2, C48.2, C57.2, C58.2, C59.2, C60.2, C61.2, C62.1, C63.2, C64.2, C65.2, C66.2, R29.1, R30.1, R31.1, R32.1, R34.1, R35.1, U$15.AGND, U$15.PGND, U7.GND, U8.GND
- net SCL: now also U7.SCL
- net SDA: now also U7.SDA
Other:
- note added: "00011101"
- note added: "3.3v LDO"
- note added: "3.6v Buck"
- note added: "I2c Adress: 1Dh"
- note added: "R29 setting Vout to 3.6v"
- note added: "This 3.1v regulator can be populated instead of using the DAC to bias the RF PA"
- moved on the sheet: U$15, U7, U8

Commit message: continued work
Parts:
- added R36, R37, R38: 5k, SparkFun-Resistors:RESISTOR0402
- added R39: DNP, SparkFun-Resistors:RESISTOR0402
Connections:
- new net N$61: R36.2, U3.A2
- new net N$62: R37.2, U3.A1
- new net N$63: R38.2, U3.A0
- new net N$64: R39.2, U6.LDAC
- new net PA_OVERTEMP_ALARM: U3.OS
- net GND: now also R36.1, R37.1, R38.1, R39.1; no longer U6.LDAC
- net PA_PWR_REF: now also U7.IN2
- net PA_PWR_SENSE: now also U7.IN3
- net PA_TEMP: now also U7.IN4
- net RF_POWER_IN: now also U7.IN0
- net RF_POWER_OUT: now also U7.IN1
Other:
- note added: "001_1101b"
- note added: "100_1000b"
- note added: "110_0000b"
- note added: "48h"
- note added: "60h"
- note removed: "00011101"
- moved on the sheet: C12, R28, U$16, U3

Commit message: Added TVS array and diode
Parts:
- removed JP1: (no value), SparkFun-Connectors:M10X2SPECIAL
- removed JP4: (no value), SparkFun-Connectors:M01PTH
- added D10, D11, D12, D13, D7: PESD5V0U5BF, RitLaunchInitiative:PESD5V0U5BF
- added R40, R41: 10k, SparkFun-Resistors:RESISTOR0402
- added U$12: DFLT13A-7, RitLaunchInitiative:DFLT13A-7
- added U$20, U$21: 10k, RitLaunchInitiative:THERMISTOR
- added X1: 679105700, con-molex:679105700
Connections:
- new net BUCK_TEMP: R40.1, U$20.1, U7.IN5
- new net PA_LOADSWITCH_TEMP: R41.1, U$21.1, U7.IN6
- net 12V: now also U$12.CATHODE
- net 3.3V: now also R40.2, R41.2; no longer JP1.1, JP1.2, JP1.3, JP1.4, JP1.6
- net 3V6_PWRGD: now also D10.P$5
- net 5V: no longer JP1.9
- net BUFF_TR_SWITCH_CTL: now also D12.P$6
- net DAC_PWR_EN: now also D7.P$1
- net DAC_PWR_FAULT: now also D10.P$1
- net GND: now also D10.P$2, D11.P$2, D12.P$2, D13.P$2, D7.P$2, U$12.ANODE, U$20.2, U$21.2; no longer JP1.10, JP1.12, JP1.5, JP1.7, JP1.8
- net N$18: now also U7.IN7; no longer JP4.1
- net N_IRQ: now also D11.P$4
- net N_SEL: now also D11.P$1
- net PA_BREAKER_OVERRIDE: now also D7.P$4
- net PA_PWR_EN: now also D7.P$3
- net PA_PWR_EN_BREAKER: now also D7.P$5
- net PA_PWR_FAULT: now also D10.P$4
- net PA_PWR_REF: now also D12.P$5
- net PA_PWR_SENSE: now also D12.P$4
- net PA_TEMP: now also D13.P$6
- net RADIO_PWR_EN: now also D7.P$6
- net RADIO_PWR_FAULT: now also D10.P$6
- net RADIO_SHUTDOWN: now also D10.P$3
- net RF_POWER_IN: now also D12.P$1
- net RF_POWER_OUT: now also D12.P$3
- net SCL: now also D13.P$1
- net SCLK: now also D11.P$5
- net SDA: now also D13.P$3
- net SDI: now also D11.P$6
- net SDO: now also D11.P$3
- net VSWR_BREAKER_STATE: now also D13.P$5
Other:
- note added: "DAC_ADC Test loop"
- note added: "I2C ADC"
- note added: "I2C Pullups"
- note added: "PA control Dac"
- note added: "PCIE MINI CARD EDGE"
- note added: "Power Sequencing Load switches"
- note added: "TVS protection arrays"
- moved on the sheet: C11, C12, C17, C18, C32, C48, C52, C53, C54, C57, C58, C59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

Commit message: finishing card edge connector
Parts:
- removed X1: 679105700, con-molex:679105700
- added U$13: RADIO_HEAD_EDGECONNECTOR, RitLaunchInitiative:RADIO_HEAD_EDGECONNECTOR
Other:
- moved on the sheet: D10, D11, D12, D13, D7, R22, R23, U$12

Commit message: added TCA9535 IO expander to simplify API if needed
Parts:
- removed C54: DNP, SparkFun-Capacitors:CAP0402-CAP
- removed D12: PESD5V0U5BF, RitLaunchInitiative:PESD5V0U5BF
- removed D3: DNP, SparkFun-LED:LED0603
- removed U$4: LP3984_DNP, RitLaunchInitiative:LP3984
- added R42, R43: 5k, SparkFun-Resistors:RESISTOR0402
- added SJ6: JUMPER-PAD-2-NOYES_SILK, SparkFun-Passives:JUMPER-PAD-2-NOYES_SILK
- added U9: TCA9535, RitLaunchInitiative:TCA9535
- C32: value DNP -> 0.1uF; device SparkFun-Capacitors:10UF-16V-10%(TANT) -> SparkFun-Capacitors:CAP0402-CAP; DIGI 399-3678-1-ND -> 311-1338-1-ND; MPN T491A105K016AT -> CC0402KRX7R7BB104
- R11: value DNP -> 5k
Connections:
- new net EXPANDER_IRQ: U$13.RESET, U9.INT
- new net N$66: R11.2, U9.A0
- new net N$67: R42.2, U9.A1
- new net N$68: R43.2, U9.A2
- net 12V: now also U$13.12V
- net 3.3V: now also C32.1, SJ6.2, U9.VCC
- net 3V1: no longer C32.+, D3.A, U$4.V_OUT
- net 3V6_PWRGD: now also U$13.DIFF_A+, U9.P06
- net 5V: no longer C54.2, U$4.VIN
- net BUFF_TR_SWITCH_CTL: now also D13.P$6, U$13.DIG_2, U9.P04; no longer D12.P$6
- net DAC_PWR_EN: now also U$13.ANALOG_1, U9.P17
- net DAC_PWR_FAULT: now also U$13.DIFF_B-, U9.P11
- net GND: now also C32.2, R42.1, R43.1, U$13.GND, U9.GND; no longer C32.-, C54.1, D12.P$2, U$4.GND
- net N$7: now also SJ6.1, U$13.3.3V; no longer D3.C, R11.2
- net N_IRQ: now also U$13.IRQ
- net N_SEL: now also U$13.SPI_CS
- net PA_BREAKER_OVERRIDE: now also U$13.ANALOG_4, U9.P14
- net PA_PWR_EN: now also U$13.ANALOG_3, U9.P15
- net PA_PWR_EN_BREAKER: now also U$13.ANALOG_5, U9.P13; no longer U$4.V_EN
- net PA_PWR_FAULT: now also U$13.DIFF_A-, U9.P07
- net PA_PWR_REF: no longer D12.P$5
- net PA_PWR_SENSE: no longer D12.P$4
- net PA_TEMP: no longer D13.P$6
- net RADIO_PWR_EN: now also U$13.ANALOG_2, U9.P16
- net RADIO_PWR_FAULT: now also U$13.DIFF_B+, U9.P10
- net RADIO_SHUTDOWN: now also U$13.DIG_1, U9.P05
- net RF_POWER_IN: no longer D12.P$1
- net RF_POWER_OUT: no longer D12.P$3
- net SCL: now also U$13.I2C_SCL, U9.SCL
- net SCLK: now also U$13.SPI_CLK
- net SDA: now also U$13.I2C_SDL, U9.SDA
- net SDI: now also U$13.SPI_MOSI
- net SDO: now also U$13.SPI_MISO
- net VSWR_BREAKER_STATE: now also U$13.ANALOG_6, U9.P12
Other:
- note added: "010_0000b"
- note added: "I2c Adress: 20h"
- note added: "Optional I0 Expander allowing module to be controlled through only i2c and SPI"
- note removed: "3.3v tollerant"
- note removed: "This 3.1v regulator can be populated instead of using the DAC to bias the RF PA"
- moved on the sheet: C12, C44, C45, C46, C47, D10, D11, D13, D7, R11, R22, R23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
