File: Electronics/TelemetryBoard/RFModule900/Design/RFModule900_Mark1.sch (EAGLE design)
At the start: 165 parts, among them T1 DC08-73, T2 DC08-73, U1 TPS2561, U2 TPS2561, U3 LM75B, U4 LTC5505, U5 LTC5505, U6 MCP4728, U7 ADC128D818, U8 MIC5504-3.3YM5, U9 TCA9535, Y1 30 Mhz

Commit message: reduced size of a couple logic gates
Parts:
- R1, R10, R11, R12, R13, R14, R15, R18, R19, R2, R20, R21, R22, R23, R24, R25, R26, R27, R28, R29, R3, R30, R31, R32, R33, R34, R35, R36, R37, R38, R39, R4, R40, R41, R42, R43, R44, R5, R6, R7, R8, R9: device SparkFun-Resistors:RESISTOR0402-RES -> SparkFun-Resistors:RESISTOR0402
- U$11, U$4, U$8: value SN74LVC1G14 -> SN74LVC1G14SOT23-56-SON; device RitLaunchInitiative:SN74LVC1G14 -> RitLaunchInitiative:SN74LVC1G14SOT23-56-SON
- U$9: value SN74LVC1G32 -> SN74LVC1G326-SON6-SON; device RitLaunchInitiative:SN74LVC1G32 -> RitLaunchInitiative:SN74LVC1G326-SON6-SON
Other:
- moved on the sheet: U$9
