File: Electronics/TelemetryBoard/RFModule900/Design/RFModule900_Mark1.brd (EAGLE design)
At the start: 100 x 30 mm, 165 parts, among them T1 DC08-73, T2 DC08-73, U1 TPS2561, U2 TPS2561, U3 LM75B, U4 LTC5505, U5 LTC5505, U6 MCP4728, U7 ADC128D818, U8 MIC5504-3.3YM5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

Commit message: adding new PCIE-36 card edge
Parts:
- added U$5: (no value), RitLaunchInitiative:PCIE_36_CARDEDGE
Changed lines of the file:
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@@
 </element>
 <element name="C54" library="SparkFun-Capacitors" package="0402-CAP" value="0.1uF" x="-17.78" y="-25.4"/>
+<element name="U$5" library="RitLaunchInitiative" package="PCIE_36_CARDEDGE" value="" x="100.33" y="15.24"/>
 </elements>
 <signals>
@@
 <contactref element="R44" pad="1"/>
 <polygon width="0.4064" layer="16">
-<vertex x="-1.27" y="30.48"/>
-<vertex x="100.33" y="30.48"/>
+<vertex x="0" y="31.75"/>
+<vertex x="100.33" y="31.75"/>
 <vertex x="100.33" y="0"/>
-<vertex x="-1.27" y="0"/>
+<vertex x="0" y="0"/>
 </polygon>
 <polygon width="0.4064" layer="2">
